File: Right/Right.kicad_pcb (KiCad board)
At the start: 2 copper layers, 169.8 x 149.7 mm, 121 parts, among them SW1 SW_PUSH, SW10 SW_PUSH, SW100 SW_Push_Dual_R, SW101 SW_Push_Dual_R, SW102 SW_Push_Dual_R, SW11 SW_PUSH, SW12 SW_PUSH, SW13 SW_PUSH, SW14 SW_PUSH, SW15 SW_PUSH, SW16 SW_PUSH, SW17 SW_PUSH, SW18 SW_PUSH, SW19 SW_PUSH, SW2 SW_PUSH, SW20 SW_PUSH, SW200 SW_SPDT, SW21 SW_PUSH, SW22 SW_PUSH, SW23 SW_PUSH, SW24 SW_PUSH, SW25 SW_PUSH, SW26 SW_PUSH, SW27 SW_PUSH, SW28 SW_PUSH, SW29 SW_PUSH, SW3 SW_PUSH, SW30 SW_PUSH, SW31 SW_PUSH, SW32 SW_PUSH, SW33 SW_PUSH, SW34 SW_PUSH, SW35 SW_PUSH, SW36 SW_PUSH, SW37 SW_PUSH, SW38 SW_PUSH, SW39 SW_PUSH, SW4 SW_PUSH, SW40 SW_PUSH, SW41 SW_PUSH, SW42 SW_PUSH, SW43 SW_PUSH, SW44 SW_PUSH, SW45 SW_PUSH, SW5 SW_PUSH, SW6 SW_PUSH, SW7 SW_PUSH, SW8 SW_PUSH, SW9 SW_PUSH, U1 CH25-2032LF, U2 CH25-2032LF

Commit message: 全体にした
Parts:
- removed D16, D17, D18, D19, D26, D27, D28, D29, D36, D37, D39, D6, D7, D8, D9: D, Diode_THT:D_DO-35_SOD27_P7.62mm_Horizontal
- removed D200, D201: D, Diode_THT:D_DO-41_SOD81_P7.62mm_Horizontal
- removed the D40 at (200.3, 150.2)
- removed the D41 at (200.3, 169.2)
- removed the D42 at (209.9, 71.8)
- removed the D43 at (217.0, 83.5)
- removed the D44 at (217.0, 112.1)
- removed the D45 at (217.8, 169.2)
- removed the REF** at (147.3, 52.2)
- removed the REF** at (172.1, 73.5)
- removed the REF** at (230.7, 78.5)
- removed the REF** at (230.7, 73.5)
- removed the REF** at (72.8, 78.6)
- removed the REF** at (72.8, 73.6)
- removed the REF** at (72.8, 52.2)
- removed the REF** at (230.7, 52.2)
- removed the REF** at (69.2, 125.2)
- removed the REF** at (154.3, 114.9)
- removed the REF** at (76.1, 188.7)
- removed the REF** at (161.9, 176.8)
- removed the REF** at (230.7, 186.3)
- removed the REF** at (230.7, 123.8)
- removed the REF** at (172.1, 78.5)
- removed SW16, SW17, SW18, SW19, SW26, SW27, SW28, SW29, SW6, SW7, SW8, SW9: SW_PUSH, keyswitches:Kailh_socket_MX
- removed SW200: SW_SPDT, mylibrary:2MS1-T1-B4-VS2-Q-E-S
- added BPM2: BleProMicro, mylibrary:BLEMicroPro, F.Cu at (295.9, 0.00)
- added C2: C, Capacitor_THT:C_Disc_D5.1mm_W3.2mm_P5.00mm, F.Cu at (312.4, 12.1)
- added D0: D, Diode_THT:D_DO-35_SOD27_P7.62mm_Horizontal, F.Cu at (20.0, 4.76)
- added D1000: D, Diode_THT:D_DO-35_SOD27_P7.62mm_Horizontal, F.Cu at (93.9, -61.4)
- added D1001: D, Diode_THT:D_DO-35_SOD27_P7.62mm_Horizontal, F.Cu at (100.4, -61.2)
- added D1002: D, Diode_THT:D_DO-35_SOD27_P7.62mm_Horizontal, F.Cu at (108.1, -61.4)
- added D1003: D, Diode_THT:D_DO-35_SOD27_P7.62mm_Horizontal, F.Cu at (270.5, 19.1)
- added D1004: D, Diode_THT:D_DO-35_SOD27_P7.62mm_Horizontal, F.Cu at (273.1, 19.1)
- added D1005: D, Diode_THT:D_DO-35_SOD27_P7.62mm_Horizontal, F.Cu at (275.6, 19.1)
- added D103: D, Diode_THT:D_DO-35_SOD27_P7.62mm_Horizontal, F.Cu at (224.8, 66.7)
- added D104: D, Diode_THT:D_DO-35_SOD27_P7.62mm_Horizontal, F.Cu at (243.8, 81.0)
- added D105: D, Diode_THT:D_DO-35_SOD27_P7.62mm_Horizontal, F.Cu at (262.9, 81.0)
- added D106: D, Diode_THT:D_DO-35_SOD27_P7.62mm_Horizontal, F.Cu at (286.7, 90.5)
- added D110: D, Diode_THT:D_DO-35_SOD27_P7.62mm_Horizontal, F.Cu at (166.3, 110.3)
- added D111: D, Diode_THT:D_DO-35_SOD27_P7.62mm_Horizontal, F.Cu at (189.3, 104.1)
- added D112: D, Diode_THT:D_DO-35_SOD27_P7.62mm_Horizontal, F.Cu at (215.3, 100.0)
- added D113: D, Diode_THT:D_DO-35_SOD27_P7.62mm_Horizontal, F.Cu at (234.3, 100.0)
- added D114: D, Diode_THT:D_DO-35_SOD27_P7.62mm_Horizontal, F.Cu at (267.7, 109.4)
- added D115: D, Diode_THT:D_DO-35_SOD27_P7.62mm_Horizontal, F.Cu at (286.7, 109.5)
- added D116: D, Diode_THT:D_DO-35_SOD27_P7.62mm_Horizontal, F.Cu at (305.8, 109.5)
- added D40 (x2): D, Diode_THT:D_DO-35_SOD27_P7.62mm_Horizontal, F.Cu at (8.10, 81.0)
- added D41 (x2): D, Diode_THT:D_DO-35_SOD27_P7.62mm_Horizontal, F.Cu at (29.5, 81.0)
- added D42: D, Diode_THT:D_DO-35_SOD27_P7.62mm_Horizontal, B.Cu at (48.6, 66.7)
- added D42: D, Diode_THT:D_DO-35_SOD27_P7.62mm_Horizontal, F.Cu at (48.6, 66.7)
- added D43 (x2): D, Diode_THT:D_DO-35_SOD27_P7.62mm_Horizontal, F.Cu at (67.6, 66.7)
- added D44 (x2): D, Diode_THT:D_DO-35_SOD27_P7.62mm_Horizontal, F.Cu at (90.5, 79.2)
- added D45 (x2): D, Diode_THT:D_DO-35_SOD27_P7.62mm_Horizontal, F.Cu at (108.9, 84.2)
- added D50: D, Diode_THT:D_DO-35_SOD27_P7.62mm_Horizontal, F.Cu at (5.71, 100.0)
- added D51: D, Diode_THT:D_DO-35_SOD27_P7.62mm_Horizontal, F.Cu at (39.1, 100.0)
- added D52: D, Diode_THT:D_DO-35_SOD27_P7.62mm_Horizontal, F.Cu at (58.1, 100.0)
- added D53: D, Diode_THT:D_DO-35_SOD27_P7.62mm_Horizontal, F.Cu at (84.2, 103.5)
- added D54: D, Diode_THT:D_DO-35_SOD27_P7.62mm_Horizontal, F.Cu at (107.2, 109.6)
- added D60: D, Diode_THT:D_DO-35_SOD27_P7.62mm_Horizontal, B.Cu at (167.6, 9.53)
- added D61: D, Diode_THT:D_DO-35_SOD27_P7.62mm_Horizontal, B.Cu at (178.3, 9.53)
- added D62: D, Diode_THT:D_DO-35_SOD27_P7.62mm_Horizontal, B.Cu at (199.6, 9.53)
- added D63: D, Diode_THT:D_DO-35_SOD27_P7.62mm_Horizontal, B.Cu at (220.9, 9.53)
- added D64: D, Diode_THT:D_DO-35_SOD27_P7.62mm_Horizontal, B.Cu at (242.2, 9.53)
- added D65: D, Diode_THT:D_DO-35_SOD27_P7.62mm_Horizontal, F.Cu at (264.8, 19.1)
- added D66: D, Diode_THT:D_DO-35_SOD27_P7.62mm_Horizontal, F.Cu at (290.8, 20.3)
- added D70: D, Diode_THT:D_DO-35_SOD27_P7.62mm_Horizontal, F.Cu at (159.0, 27.2)
- added D71: D, Diode_THT:D_DO-35_SOD27_P7.62mm_Horizontal, B.Cu at (188.9, 9.53)
- added D72: D, Diode_THT:D_DO-35_SOD27_P7.62mm_Horizontal, B.Cu at (210.3, 9.53)
- added D73: D, Diode_THT:D_DO-35_SOD27_P7.62mm_Horizontal, B.Cu at (231.6, 9.53)
- added D74: D, Diode_THT:D_DO-35_SOD27_P7.62mm_Horizontal, B.Cu at (252.9, 9.53)
- added D75: D, Diode_THT:D_DO-35_SOD27_P7.62mm_Horizontal, F.Cu at (262.9, 23.8)
- added D76: D, Diode_THT:D_DO-35_SOD27_P7.62mm_Horizontal, F.Cu at (281.9, 23.8)
- added D77: D, Diode_THT:D_DO-35_SOD27_P7.62mm_Horizontal, F.Cu at (303.4, 23.8)
- added D80: D, Diode_THT:D_DO-35_SOD27_P7.62mm_Horizontal, F.Cu at (154.7, 48.0)
- added D81: D, Diode_THT:D_DO-35_SOD27_P7.62mm_Horizontal, F.Cu at (173.1, 43.1)
- added D82: D, Diode_THT:D_DO-35_SOD27_P7.62mm_Horizontal, F.Cu at (196.2, 28.6)
- added D83: D, Diode_THT:D_DO-35_SOD27_P7.62mm_Horizontal, F.Cu at (215.3, 28.6)
- added D84: D, Diode_THT:D_DO-35_SOD27_P7.62mm_Horizontal, F.Cu at (234.3, 28.6)
- added D85: D, Diode_THT:D_DO-35_SOD27_P7.62mm_Horizontal, F.Cu at (253.4, 42.9)
- added D86: D, Diode_THT:D_DO-35_SOD27_P7.62mm_Horizontal, F.Cu at (272.4, 42.9)
- added D87: D, Diode_THT:D_DO-35_SOD27_P7.62mm_Horizontal, F.Cu at (303.4, 52.4)
- added D90: D, Diode_THT:D_DO-35_SOD27_P7.62mm_Horizontal, F.Cu at (155.0, 67.7)
- added D91: D, Diode_THT:D_DO-35_SOD27_P7.62mm_Horizontal, F.Cu at (173.4, 62.7)
- added D92: D, Diode_THT:D_DO-35_SOD27_P7.62mm_Horizontal, F.Cu at (201.0, 47.6)
- added D93: D, Diode_THT:D_DO-35_SOD27_P7.62mm_Horizontal, F.Cu at (224.8, 47.6)
- added D94: D, Diode_THT:D_DO-35_SOD27_P7.62mm_Horizontal, F.Cu at (243.8, 61.9)
- added D95: D, Diode_THT:D_DO-35_SOD27_P7.62mm_Horizontal, F.Cu at (262.9, 61.9)
- added D96: D, Diode_THT:D_DO-35_SOD27_P7.62mm_Horizontal, F.Cu at (281.9, 66.7)
- added DD1: D, Diode_THT:D_DO-41_SOD81_P7.62mm_Horizontal, F.Cu at (36.5, -68.1)
- added DD2: D, Diode_THT:D_DO-41_SOD81_P7.62mm_Horizontal, F.Cu at (69.6, -69.7)
- added DD3: D, Diode_THT:D_DO-41_SOD81_P7.62mm_Horizontal, F.Cu at (168.3, 20.3)
- added DD4: D, Diode_THT:D_DO-41_SOD81_P7.62mm_Horizontal, F.Cu at (168.3, 15.2)
- added LED2: LED, LED_THT:LED_D3.0mm, F.Cu at (303.5, -14.0)
- added R2: R, Resistor_THT:R_Axial_DIN0204_L3.6mm_D1.6mm_P7.62mm_Horizontal, F.Cu at (306.1, -10.2)
- added REF**: Spacer, mylibrary:Spacer, F.Cu at (233.7, -7.53)
- added REF**: Spacer, mylibrary:Spacer, F.Cu at (258.4, 13.8)
- added REF**: Spacer, mylibrary:Spacer, F.Cu at (317.1, 18.8)
- added REF**: Spacer, mylibrary:Spacer, F.Cu at (317.1, 13.8)
- added REF**: Spacer, mylibrary:Spacer, F.Cu at (159.2, 18.9)
- added REF**: Spacer, mylibrary:Spacer, F.Cu at (159.2, 13.9)
- added REF**: Spacer, mylibrary:Spacer, F.Cu at (159.2, -7.53)
- added REF**: Spacer, mylibrary:Spacer, F.Cu at (317.1, -7.53)
- added REF**: Spacer, mylibrary:Spacer, F.Cu at (155.5, 65.5)
- added REF**: Spacer, mylibrary:Spacer, F.Cu at (240.7, 55.2)
- added REF**: Spacer, mylibrary:Spacer, F.Cu at (162.5, 129.0)
- added REF**: Spacer, mylibrary:Spacer, F.Cu at (248.3, 117.1)
- added REF**: Spacer, mylibrary:Spacer, F.Cu at (317.1, 126.6)
- added REF**: Spacer, mylibrary:Spacer, F.Cu at (317.1, 64.1)
- added REF**: Spacer, mylibrary:Spacer, F.Cu at (258.4, 18.8)
- added SW0: SW_PUSH, keyswitches:Kailh_socket_MX, F.Cu at (23.8, 14.3)
- added SW1000: SW_Push_Dual_R, Button_Switch_THT:SW_TH_Tactile_Omron_B3F-10xx, F.Cu at (57.7, -26.3)
- added SW1001: SW_Push_Dual_R, Button_Switch_THT:SW_TH_Tactile_Omron_B3F-10xx, F.Cu at (41.2, -24.4)
- added SW1002: SW_Push_Dual_R, Button_Switch_THT:SW_TH_Tactile_Omron_B3F-10xx, F.Cu at (69.6, -27.1)
- added SW1003: SW_Push_Dual_R, Button_Switch_THT:SW_TH_Tactile_Omron_B3F-10xx, F.Cu at (278.1, -12.0)
- added SW1004: SW_Push_Dual_R, Button_Switch_THT:SW_TH_Tactile_Omron_B3F-10xx, F.Cu at (287.0, -12.0)
- added SW1005: SW_Push_Dual_R, Button_Switch_THT:SW_TH_Tactile_Omron_B3F-10xx, F.Cu at (295.9, -12.1)
- added SW103: SW_PUSH, keyswitches:Kailh_socket_MX, F.Cu at (228.6, 76.2)
- added SW104: SW_PUSH, keyswitches:Kailh_socket_MX, F.Cu at (247.7, 90.5)
- added SW105: SW_PUSH, keyswitches:Kailh_socket_MX, F.Cu at (266.7, 90.5)
- added SW106: SW_PUSH, keyswitches:Kailh_socket_MX, F.Cu at (290.5, 100.0)
- added SW110: SW_PUSH, keyswitches:Kailh_socket_MX, F.Cu at (172.4, 118.5)
- added SW111: SW_PUSH, keyswitches:Kailh_socket_MX, F.Cu at (195.4, 112.4)
- added SW112: SW_PUSH, keyswitches:Kailh_socket_MX, F.Cu at (219.1, 109.5)
- added SW113: SW_PUSH, keyswitches:Kailh_socket_MX, F.Cu at (238.1, 109.5)
- added SW114: SW_PUSH, keyswitches:Kailh_socket_MX, F.Cu at (271.5, 119.1)
- added SW115: SW_PUSH, keyswitches:Kailh_socket_MX, F.Cu at (290.5, 119.1)
- added SW116: SW_PUSH, keyswitches:Kailh_socket_MX, F.Cu at (309.6, 119.1)
- added SW50: SW_PUSH, keyswitches:Kailh_socket_MX, F.Cu at (9.53, 109.5)
- added SW51: SW_PUSH, keyswitches:Kailh_socket_MX, F.Cu at (42.9, 109.5)
- added SW52: SW_PUSH, keyswitches:Kailh_socket_MX, F.Cu at (61.9, 109.5)
- added SW53: SW_PUSH, keyswitches:Kailh_socket_MX, F.Cu at (85.4, 113.7)
- added SW54: SW_PUSH, keyswitches:Kailh_socket_MX, F.Cu at (108.4, 119.8)
- added SW60: SW_PUSH, keyswitches:Kailh_socket_MX, F.Cu at (166.7, 0.00)
- added SW61: SW_PUSH, keyswitches:Kailh_socket_MX, F.Cu at (185.7, 0.00)
- added SW62: SW_PUSH, keyswitches:Kailh_socket_MX, F.Cu at (204.8, 0.00)
- added SW63: SW_PUSH, keyswitches:Kailh_socket_MX, F.Cu at (223.8, 0.00)
- added SW64: SW_PUSH, keyswitches:Kailh_socket_MX, F.Cu at (242.9, 0.00)
- added SW65: SW_PUSH, keyswitches:Kailh_socket_MX, F.Cu at (261.9, 0.00)
- added SW66: SW_PUSH, keyswitches:Kailh_socket_MX, F.Cu at (281.0, 0.00)
- added SW70: SW_PUSH, keyswitches:Kailh_socket_MX, F.Cu at (165.1, 35.4)
- added SW71: SW_PUSH, keyswitches:Kailh_socket_MX, F.Cu at (190.5, 19.1)
- added SW72: SW_PUSH, keyswitches:Kailh_socket_MX, F.Cu at (209.6, 19.1)
- added SW73: SW_PUSH, keyswitches:Kailh_socket_MX, F.Cu at (228.6, 19.1)
- added SW74: SW_PUSH, keyswitches:Kailh_socket_MX, F.Cu at (247.7, 19.1)
- added SW75: SW_PUSH, keyswitches:Kailh_socket_MX, F.Cu at (266.7, 33.3)
- added SW76: SW_PUSH, keyswitches:Kailh_socket_MX, F.Cu at (285.8, 33.3)
- added SW77: SW_PUSH, keyswitches:Kailh_socket_MX, F.Cu at (307.2, 33.3)
- added SW80: SW_PUSH, keyswitches:Kailh_socket_MX, F.Cu at (160.8, 56.3)
- added SW81: SW_PUSH, keyswitches:Kailh_socket_MX, F.Cu at (179.2, 51.3)
- added SW82: SW_PUSH, keyswitches:Kailh_socket_MX, F.Cu at (200.0, 38.1)
- added SW83: SW_PUSH, keyswitches:Kailh_socket_MX, F.Cu at (219.1, 38.1)
- added SW84: SW_PUSH, keyswitches:Kailh_socket_MX, F.Cu at (238.1, 38.1)
- added SW85: SW_PUSH, keyswitches:Kailh_socket_MX, F.Cu at (257.2, 52.4)
- added SW86: SW_PUSH, keyswitches:Kailh_socket_MX, F.Cu at (276.2, 52.4)
- added SW87: SW_PUSH, keyswitches:Kailh_socket_MX, F.Cu at (307.2, 61.9)
- added SW90: SW_PUSH, keyswitches:Kailh_socket_MX, F.Cu at (161.2, 75.9)
- added SW91: SW_PUSH, keyswitches:Kailh_socket_MX, F.Cu at (179.6, 71.0)
- added SW92: SW_PUSH, keyswitches:Kailh_socket_MX, F.Cu at (204.8, 57.1)
- added SW93: SW_PUSH, keyswitches:Kailh_socket_MX, F.Cu at (228.6, 57.1)
- added SW94: SW_PUSH, keyswitches:Kailh_socket_MX, F.Cu at (247.7, 71.4)
- added SW95: SW_PUSH, keyswitches:Kailh_socket_MX, F.Cu at (266.7, 71.4)
- added SW96: SW_PUSH, keyswitches:Kailh_socket_MX, F.Cu at (285.8, 76.2)
- added SWITCH0: SW_SPDT, mylibrary:2MS1-T1-B4-VS2-Q-E-S, F.Cu at (14.8, -72.2)
- added SWITCH1: SW_SPDT, mylibrary:2MS1-T1-B4-VS2-Q-E-S, F.Cu at (312.4, -14.0)
- added U3: CH25-2032LF, CH25-2032LF:CH252032LF, F.Cu at (213.4, 3.17)
- added U4: CH25-2032LF, CH25-2032LF:CH252032LF, F.Cu at (175.3, 3.18)
- SW100, SW101, SW102: value SW_Push_Dual_R -> SW_PUSH; footprint Button_Switch_THT:SW_TH_Tactile_Omron_B3F-10xx -> keyswitches:Kailh_socket_MX
- moved C1 247.8 mm to (14.1, -56.5)
- moved R1 228.8 mm to (7.97, -37.1)
- moved LED1 217.6 mm to (13.3, -30.5)
- moved SW40 204.3 mm to (11.9, 90.5)
- moved BPM1 197.4 mm to (21.8, -1.44), turned to 90 degrees
- moved SW41 192.3 mm to (33.3, 90.5)
- moved D30 171.2 mm to (8.10, 61.9), turned to 0 degrees
- moved SW30 164.1 mm to (11.9, 71.4)
- moved SW42 162.1 mm to (52.4, 76.2)
- moved D12 160.7 mm to (58.1, 9.53), turned to 0 degrees
- moved SW12 160.1 mm to (61.9, 19.1), turned to 0 degrees
- moved D5 158.4 mm to (115.3, -9.53), turned to 0 degrees
- moved SW5 156.6 mm to (119.1, 0.00), turned to 0 degrees
- moved SW43 150.3 mm to (71.4, 76.2)
- moved D31 148.6 mm to (29.5, 61.9)
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Connections:
- net bat renamed bat0
- net gnd renamed gnd0
- net led renamed led0
- BPM1 pad 12: col6 -> Net-(BPM1-Pad12)
- BPM1 pad 13: col7 -> Net-(BPM1-Pad13)
- BPM1 pad 14: rowsys -> rowsys0
- D10 pad 1: row3 -> row1
- D100 pad 1: rowsys -> row10
- D101 pad 1: rowsys -> row10
- D102 pad 1: rowsys -> row10
- D11 pad 1: row4 -> row1
- D12 pad 1: row5 -> row1
- D13 pad 1: row0 -> row1
- D15 pad 1: row2 -> row1
- D2 pad 1: row1 -> row0
- D20 pad 1: row1 -> row2
- D22 pad 1: row3 -> row2
- D23 pad 1: row4 -> row2
- D24 pad 1: row5 -> row2
- D25 pad 1: row0 -> row2
- D3 pad 1: row2 -> row0
- D30 pad 1: row0 -> row3
- D31 pad 1: row1 -> row3
- D32 pad 1: row2 -> row3
- D34 pad 1: row4 -> row3
- D35 pad 1: row5 -> row3
- D38 pad 1: row2 -> row8
- D4 pad 1: row3 -> row0
- D5 pad 1: row4 -> row0
- SW1 pad 1: col0 -> col1
- SW10 pad 1: col1 -> col0
- SW100 pad 1: col5 -> col6
- SW100 pad 2: Net-(SW100-Pad2) -> Net-(D100-Pad2)
- SW101 pad 1: col6 -> col7
- SW101 pad 2: Net-(SW101-Pad2) -> Net-(D101-Pad2)
- SW102 pad 1: col7 -> col8
- SW102 pad 2: Net-(SW102-Pad2) -> Net-(D102-Pad2)
- SW12 pad 1: col1 -> col2
- SW13 pad 1: col2 -> col3
- SW14 pad 1: col2 -> col4
- SW15 pad 1: col2 -> col5
- SW2 pad 1: col0 -> col2
- SW20 pad 1: col3 -> col0
- SW21 pad 1: col3 -> col1
- SW22 pad 1: col3 -> col2
- SW24 pad 1: col3 -> col4
- SW25 pad 1: col4 -> col5
- SW3 pad 1: col0 -> col3
- SW30 pad 1: col5 -> col0
- SW31 pad 1: col5 -> col1
- SW32 pad 1: col5 -> col2
- SW33 pad 1: col5 -> col3
- SW34 pad 1: col5 -> col4
- SW36 pad 1: col6 -> col12
- SW37 pad 1: col6 -> col12
- SW38 pad 1: col6 -> col12
- SW39 pad 1: col6 -> col12
- SW4 pad 1: col0 -> col4
- SW40 pad 1: col6 -> col0
- SW41 pad 1: col6 -> col1
- SW42 pad 1: col7 -> col2
- SW43 pad 1: col7 -> col3
- SW44 pad 1: col7 -> col4
- SW45 pad 1: col7 -> col5
- SW5 pad 1: col0 -> col5
Routing:
- net col0: track 387.7 -> 0.00 mm
- net col1: track 349.9 -> 0.00 mm
- net col8: track 0.00 -> 331.1 mm
- net col2: track 331.1 -> 0.00 mm
- net col9: track 0.00 -> 308.4 mm
- net col3: track 308.4 -> 0.00 mm
- net col4: track 288.7 -> 0.00 mm
- net col10: track 0.00 -> 288.7 mm
- net row11: track 0.00 -> 272.2 mm
- net row5: track 272.2 -> 0.00 mm
- net row4: track 261.5 -> 0.00 mm
- net row10: track 0.00 -> 261.5 mm
- net row9: track 0.00 -> 242.1 mm
- net row3: track 242.1 -> 0.00 mm
- net row2: track 225.3 -> 0.00 mm
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