File: Right/Right.kicad_pcb (KiCad board)
At the start: 2 copper layers, 169.8 x 149.7 mm, 215 parts, among them SW0 SW_PUSH, SW1 SW_PUSH, SW10 SW_PUSH, SW100 SW_PUSH, SW1000 SW_Push_Dual_R, SW1001 SW_Push_Dual_R, SW1002 SW_Push_Dual_R, SW1003 SW_Push_Dual_R, SW1004 SW_Push_Dual_R, SW1005 SW_Push_Dual_R, SW101 SW_PUSH, SW102 SW_PUSH, SW103 SW_PUSH, SW104 SW_PUSH, SW105 SW_PUSH, SW106 SW_PUSH, SW11 SW_PUSH, SW110 SW_PUSH, SW111 SW_PUSH, SW112 SW_PUSH, SW113 SW_PUSH, SW114 SW_PUSH, SW115 SW_PUSH, SW116 SW_PUSH, SW12 SW_PUSH, SW13 SW_PUSH, SW14 SW_PUSH, SW15 SW_PUSH, SW2 SW_PUSH, SW20 SW_PUSH, SW21 SW_PUSH, SW22 SW_PUSH, SW23 SW_PUSH, SW24 SW_PUSH, SW25 SW_PUSH, SW3 SW_PUSH, SW30 SW_PUSH, SW31 SW_PUSH, SW32 SW_PUSH, SW33 SW_PUSH, SW34 SW_PUSH, SW35 SW_PUSH, SW36 SW_PUSH, SW37 SW_PUSH, SW38 SW_PUSH, SW39 SW_PUSH, SW4 SW_PUSH, SW40 SW_PUSH, SW41 SW_PUSH, SW42 SW_PUSH, SW43 SW_PUSH, SW44 SW_PUSH, SW45 SW_PUSH, SW5 SW_PUSH, SW50 SW_PUSH, SW51 SW_PUSH, SW52 SW_PUSH, SW53 SW_PUSH, SW54 SW_PUSH, SW60 SW_PUSH, SW61 SW_PUSH, SW62 SW_PUSH, SW63 SW_PUSH, SW64 SW_PUSH, SW65 SW_PUSH, SW66 SW_PUSH, SW70 SW_PUSH, SW71 SW_PUSH, SW72 SW_PUSH, SW73 SW_PUSH, SW74 SW_PUSH, SW75 SW_PUSH, SW76 SW_PUSH, SW77 SW_PUSH, SW80 SW_PUSH, SW81 SW_PUSH, SW82 SW_PUSH, SW83 SW_PUSH, SW84 SW_PUSH, SW85 SW_PUSH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

Commit message: なんか
Parts:
- moved BPM1 91.2 mm to (113.0, -0.20)
Changed lines of the file:
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@@
   )
   (module mylibrary:BLEMicroPro (layer F.Cu)
-    (at 21.81 -1.44 90)
+    (at 113.04 -0.2 90)
     (fp_text reference BPM1 (at -0.136 -0.812 180) (layer F.SilkS) hide
       (effects (font (size 1 1) (thickness 0.15)))

Commit message: 途中
Parts:
- moved BPM2 115.6 mm to (180.3, 0.00), turned to 90 degrees
- moved DD3 95.5 mm to (245.8, -35.6)
- moved DD4 95.5 mm to (245.7, -40.6)
- moved C2 48.4 mm to (287.4, -29.4)
- moved U4 34.0 mm to (179.1, -30.6)
- moved U3 31.5 mm to (213.1, -28.3)
- moved SW1003 28.0 mm to (298.5, 7.24)
- moved SW1004 28.0 mm to (307.4, 7.24)
- moved SW1005 28.0 mm to (316.3, 7.18)
- moved D71 10.8 mm to (179.1, 14.0), turned to 270 degrees
- moved SWITCH1 10.5 mm to (309.9, -3.81)
- moved LED2 10.2 mm to (302.3, -3.81)
- moved D80 9.53 mm to (163.9, 45.6)
- moved D60 8.91 mm to (158.8, 10.2)
- moved D61 8.14 mm to (170.2, 10.2)
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Routing:
- net col6: track 387.7 -> 98.3 mm
- net col7: track 349.9 -> 105.0 mm
- net col8: track 331.1 -> 126.2 mm
- net Net-(DD3-Pad1): track 192.7 -> 0.00 mm
- net col9: track 308.4 -> 128.7 mm
- net col10: track 288.7 -> 115.0 mm
- net row11: track 272.2 -> 145.4 mm
- net row10: track 261.5 -> 146.5 mm
- net row9: track 242.1 -> 139.9 mm
- net row7: track 205.1 -> 108.7 mm
- net Net-(DD3-Pad2): track 94.8 -> 0.00 mm
- net col13: track 171.6 -> 88.6 mm
- net row6: track 170.0 -> 100.9 mm
- net row8: track 225.3 -> 159.2 mm
- net col11: track 189.8 -> 139.0 mm
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
Commit message: 途中
Parts:
- moved D60 20.0 mm to (177.3, 17.8), turned to 180 degrees
- moved D70 19.4 mm to (177.3, 20.8), turned to 180 degrees
- moved D61 13.2 mm to (183.4, 10.2)
- moved D80 5.24 mm to (169.0, 44.3)
- moved D81 2.68 mm to (180.3, 41.4)
- moved D71 1.27 mm to (179.8, 13.0)
Connections:
- BPM1 pad 16: row0 -> row5
- BPM1 pad 17: row1 -> row4
- BPM1 pad 18: row2 -> row3
- BPM1 pad 19: row3 -> row2
- BPM1 pad 20: row4 -> row1
- BPM1 pad 21: row5 -> row0
- BPM2 pad 10: col10 -> row7
- BPM2 pad 11: col11 -> row6
- BPM2 pad 12: col12 -> led1
- BPM2 pad 13: col13 -> rowsys1
- BPM2 pad 14: rowsys1 -> col13
- BPM2 pad 15: led1 -> col12
- BPM2 pad 16: row6 -> col11
- BPM2 pad 17: row7 -> col10
- BPM2 pad 18: row8 -> col9
- BPM2 pad 19: row9 -> col8
- BPM2 pad 20: row10 -> col7
- BPM2 pad 21: row11 -> col6
- BPM2 pad 6: col6 -> row11
- BPM2 pad 7: col7 -> row10
- BPM2 pad 8: col8 -> row9
- BPM2 pad 9: col9 -> row8
Routing:
- net row11: track 145.4 -> 275.2 mm
- net row10: track 146.5 -> 250.4 mm
- net row9: track 139.9 -> 218.1 mm
- net row8: track 159.2 -> 209.5 mm
- net col7: track 105.0 -> 149.9 mm
- net col6: track 98.3 -> 141.9 mm
- net col8: track 126.2 -> 165.6 mm
- net row7: track 108.7 -> 143.6 mm
- net row6: track 100.9 -> 132.1 mm
- net Net-(D61-Pad2): track 0.00 -> 27.4 mm
- net Net-(D60-Pad2): track 0.00 -> 24.7 mm
- net Net-(D70-Pad2): track 13.5 -> 19.2 mm
- net Net-(D80-Pad2): track 23.4 -> 29.0 mm
- net Net-(D71-Pad2): track 0.00 -> 5.35 mm
- net Net-(D81-Pad2): track 18.3 -> 21.1 mm

Commit message: とりあえず右手全部つながった
Parts:
- moved C2 129.3 mm to (165.1, 12.7), turned to 0 degrees
- moved DD4 66.6 mm to (281.9, 15.2), turned to 180 degrees
- moved U3 66.1 mm to (271.8, 2.29), turned to 270 degrees
- moved U4 63.7 mm to (233.7, 2.29), turned to 270 degrees
- moved DD3 59.3 mm to (281.9, 11.4), turned to 180 degrees
- moved D1003 35.1 mm to (305.6, 19.1)
- moved D1005 35.1 mm to (310.6, 19.1)
- moved D1004 35.1 mm to (308.1, 19.1)
- moved R2 22.0 mm to (301.8, 11.4), turned to 270 degrees
- moved REF** 18.7 mm to (252.4, -7.53)
- moved D81 1.15 mm to (179.2, 41.5)
- moved D62 1.06 mm to (200.7, 9.53)
- moved D72 0.85 mm to (211.1, 9.53)
- moved D63 0.64 mm to (221.5, 9.53)
- moved D73 0.42 mm to (232.0, 9.53)
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Connections:
- BPM2 pad 14: col13 -> col8
- BPM2 pad 15: col12 -> col9
- BPM2 pad 16: col11 -> col10
- BPM2 pad 17: col10 -> col11
- BPM2 pad 18: col9 -> col12
- BPM2 pad 19: col8 -> col13
Routing:
- net col13: track 88.6 -> 364.4 mm
- net col12: track 132.2 -> 398.6 mm
- net col11: track 139.0 -> 380.1 mm
- net col10: track 115.0 -> 302.6 mm
- net bat1: track 0.00 -> 171.8 mm
- net col9: track 128.7 -> 291.8 mm
- net rowsys1: track 5.08 -> 130.2 mm
- net led1: track 0.00 -> 123.0 mm
- net Net-(DD4-Pad2): track 0.00 -> 66.0 mm
- net Net-(DD3-Pad1): track 0.00 -> 40.1 mm
- net row7: track 143.6 -> 180.4 mm
- net Net-(DD3-Pad2): track 0.00 -> 26.3 mm
- net Net-(LED2-Pad2): track 0.00 -> 18.1 mm
- net row6: track 132.1 -> 148.3 mm
- net Net-(D61-Pad2): track 27.4 -> 13.7 mm
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Other:
- board size 169.8 x 149.7 mm -> 169.8 x 140.8 mm

Commit message: fix
Parts:
- removed D38: D, Diode_THT:D_DO-35_SOD27_P7.62mm_Horizontal
- removed the D40 at (8.10, 81.0)
- removed the D41 at (29.5, 81.0)
- removed the D42 at (48.6, 66.7)
- removed the D43 at (67.6, 66.7)
- removed the D44 at (90.5, 79.2)
- removed the D45 at (108.9, 84.2)
- removed SW36, SW37, SW38, SW39: SW_PUSH, keyswitches:Kailh_socket_MX
- moved D4 1.12 mm to (96.2, -10.7)
- moved D5 0.76 mm to (115.3, -10.3)
Routing:
- net Net-(D76-Pad2): track 0.00 -> 14.3 mm
- net Net-(D37-Pad2): track 14.3 -> 0.00 mm
- net col9: track 291.8 -> 292.5 mm

Commit message: fix
Routing:
- net row8: track 199.5 -> 209.2 mm

Commit message: 右手で来た
Routing:
- net gnd1: track 0.00 -> 66.0 mm
- net bat1: track 171.8 -> 178.6 mm
Changed lines of the file:
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@@
     (thickness 1.6)
     (drawings 34)
-    (tracks 556)
+    (tracks 561)
     (zones 0)
     (modules 204)
@@
   )
   (setup
-    (last_trace_width 0.25)
+    (last_trace_width 0.5)
     (user_trace_width 0.5)
     (trace_clearance 0.2)
@@
   (segment (start 208.975 66.675) (end 213.36 66.675) (width 0.25) (layer B.Cu) (net 52))
   (segment (start 201.99 73.66) (end 208.975 66.675) (width 0.25) (layer B.Cu) (net 52))
+  (segment (start 216.621101 -8.832401) (end 173.932001 -8.832401) (width 0.5) (layer B.Cu) (net 61))
+  (segment (start 223.009601 -2.443901) (end 216.621101 -8.832401) (width 0.5) (layer B.Cu) (net 61))
+  (segment (start 173.932001 -8.832401) (end 172.72 -7.6204) (width 0.5) (layer B.Cu) (net 61))
+  (segment (start 228.926099 -2.443901) (end 223.009601 -2.443901) (width 0.5) (layer B.Cu) (net 61))
+  (segment (start 233.66 2.29) (end 228.926099 -2.443901) (width 0.5) (layer B.Cu) (net 61))
   (segment (start 215.84 23.495) (end 206.315 33.02) (width 0.25) (layer B.Cu) (net 62))
   (segment (start 215.84 13.97) (end 215.84 23.495) (width 0.25) (layer B.Cu) (net 62))
@@
   (segment (start 163.222345 81.365255) (end 158.660186 76.803096) (width 0.25) (layer F.Cu) (net 75))
   (segment (start 170.88395 108.243003) (end 163.222345 100.581398) (width 0.25) (layer F.Cu) (net 75))
-  (segment (start 174.678239 -8.832401) (end 173.932001 -8.086163) (width 0.5) (layer F.Cu) (net 79))
-  (segment (start 169.76 4.66) (end 165.52 4.66) (width 0.5) (layer F.Cu) (net 79))
-  (segment (start 248.811097 -8.832401) (end 174.678239 -8.832401) (width 0.5) (layer F.Cu) (net 79))
-  (segment (start 253.156501 -5.974999) (end 251.668499 -5.974999) (width 0.5) (layer F.Cu) (net 79))
-  (segment (start 307.960999 -8.269001) (end 255.450503 -8.269001) (width 0.5) (layer F.Cu) (net 79))
+  (segment (start 162.56 10.16) (end 165.1 12.7) (width 0.5) (layer F.Cu) (net 79))
+  (segment (start 162.56 7.62) (end 162.56 10.16) (width 0.5) (layer F.Cu) (net 79))
+  (segment (start 160.306599 5.366599) (end 162.56 7.62) (width 0.5) (layer F.Cu) (net 79))
+  (segment (start 160.712501 -1.030335) (end 160.306599 -0.624433) (width 0.5) (layer F.Cu) (net 79))
+  (segment (start 160.306599 -0.624433) (end 160.306599 5.366599) (width 0.5) (layer F.Cu) (net 79))
+  (segment (start 160.712501 -7.566263) (end 160.712501 -1.030335) (width 0.5) (layer F.Cu) (net 79))
+  (segment (start 161.978639 -8.832401) (end 160.712501 -7.566263) (width 0.5) (layer F.Cu) (net 79))
   (segment (start 251.668499 -5.974999) (end 248.811097 -8.832401) (width 0.5) (layer F.Cu) (net 79))
-  (segment (start 173.932001 0.487999) (end 169.76 4.66) (width 0.5) (layer F.Cu) (net 79))
-  (segment (start 173.932001 -8.086163) (end 173.932001 0.487999) (width 0.5) (layer F.Cu) (net 79))
+  (segment (start 253.156501 -5.974999) (end 251.668499 -5.974999) (width 0.5) (layer F.Cu) (net 79))
   (segment (start 255.450503 -8.269001) (end 253.156501 -5.974999) (width 0.5) (layer F.Cu) (net 79))
-  (segment (start 165.52 4.66) (end 162.56 7.62) (width 0.5) (layer F.Cu) (net 79))
+  (segment (start 307.960999 -8.269001) (end 255.450503 -8.269001) (width 0.5) (layer F.Cu) (net 79))
+  (segment (start 248.811097 -8.832401) (end 161.978639 -8.832401) (width 0.5) (layer F.Cu) (net 79))
   (segment (start 312.42 -3.81) (end 307.960999 -8.269001) (width 0.5) (layer F.Cu) (net 79))
-  (segment (start 162.56 10.16) (end 165.1 12.7) (width 0.5) (layer F.Cu) (net 79))
-  (segment (start 162.56 7.62) (end 162.56 10.16) (width 0.5) (layer F.Cu) (net 79))
   (segment (start 159.1275 9.5215) (end 159.1275 -2.54) (width 0.25) (layer B.Cu) (net 86))
   (segment (start 167.386 17.78) (end 159.1275 9.5215) (width 0.25) (layer B.Cu) (net 86))

Commit message: 左手調整中
Parts:
- added REF**: Spacer, mylibrary:Spacer, F.Cu at (2.00, 121.8)
- added REF**: Spacer, mylibrary:Spacer, F.Cu at (118.5, 129.0)
- moved D106 4.76 mm to (286.7, 85.7)
- moved REF** 4.76 mm to (317.1, 121.8)
- moved SW106 4.76 mm to (290.5, 95.2)
- moved SW114 4.76 mm to (271.5, 114.3)
- moved SW115 4.76 mm to (290.5, 114.3)
- moved SW116 4.76 mm to (309.6, 114.3)
- moved SW50 4.76 mm to (9.53, 114.3)
- moved SW96 4.76 mm to (285.8, 71.4)
- moved D96 4.76 mm to (281.9, 61.9)
- moved D114 4.76 mm to (267.7, 104.6)
- moved D115 4.76 mm to (286.7, 104.8)
- moved D116 4.76 mm to (305.8, 104.8)
- moved SW54 1.33 mm to (108.6, 118.5)
- moved SW53 1.33 mm to (85.6, 112.4)
Routing:
- net col12: track 398.6 -> 387.8 mm
- net col13: track 364.4 -> 353.7 mm
- net row10: track 250.4 -> 243.4 mm
- net row11: track 275.2 -> 272.3 mm
- net col11: track 380.1 -> 377.3 mm
- net row9: track 218.6 -> 217.5 mm
Other:
- board size 169.8 x 140.8 mm -> 356.7 x 140.8 mm
