File: Right/Right.kicad_pcb (KiCad board)
At the start: 2 copper layers, 316.7 x 290.8 mm, 213 parts, among them SW0 SW_PUSH, SW1 SW_PUSH, SW10 SW_PUSH, SW100 SW_PUSH, SW1000 SW_Push_Dual_R, SW1001 SW_Push_Dual_R, SW1002 SW_Push_Dual_R, SW1003 SW_Push_Dual_R, SW1004 SW_Push_Dual_R, SW1005 SW_Push_Dual_R, SW101 SW_PUSH, SW102 SW_PUSH, SW103 SW_PUSH, SW104 SW_PUSH, SW105 SW_PUSH, SW106 SW_PUSH, SW11 SW_PUSH, SW110 SW_PUSH, SW111 SW_PUSH, SW112 SW_PUSH, SW113 SW_PUSH, SW114 SW_PUSH, SW115 SW_PUSH, SW116 SW_PUSH, SW12 SW_PUSH, SW13 SW_PUSH, SW14 SW_PUSH, SW15 SW_PUSH, SW2 SW_PUSH, SW20 SW_PUSH, SW21 SW_PUSH, SW22 SW_PUSH, SW23 SW_PUSH, SW24 SW_PUSH, SW25 SW_PUSH, SW3 SW_PUSH, SW30 SW_PUSH, SW31 SW_PUSH, SW32 SW_PUSH, SW33 SW_PUSH, SW34 SW_PUSH, SW35 SW_PUSH, SW4 SW_PUSH, SW40 SW_PUSH, SW41 SW_PUSH, SW42 SW_PUSH, SW43 SW_PUSH, SW44 SW_PUSH, SW45 SW_PUSH, SW5 SW_PUSH, SW50 SW_PUSH, SW51 SW_PUSH, SW52 SW_PUSH, SW53 SW_PUSH, SW54 SW_PUSH, SW60 SW_PUSH, SW61 SW_PUSH, SW62 SW_PUSH, SW63 SW_PUSH, SW64 SW_PUSH, SW65 SW_PUSH, SW66 SW_PUSH, SW70 SW_PUSH, SW71 SW_PUSH, SW72 SW_PUSH, SW73 SW_PUSH, SW74 SW_PUSH, SW75 SW_PUSH, SW76 SW_PUSH, SW77 SW_PUSH, SW80 SW_PUSH, SW81 SW_PUSH, SW82 SW_PUSH, SW83 SW_PUSH, SW84 SW_PUSH, SW85 SW_PUSH, SW86 SW_PUSH, SW87 SW_PUSH, SW90 SW_PUSH, SW91 SW_PUSH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

Commit message: 右手トッププレート
Parts:
- added REF**: Spacer, mylibrary:Spacer, F.Cu at (240.7, 205.2)
- added REF**: Spacer, mylibrary:Spacer, F.Cu at (156.0, 217.4)
- added REF**: Spacer, mylibrary:Spacer, F.Cu at (317.1, 254.8)
- added REF**: Spacer, mylibrary:Spacer, F.Cu at (317.1, 175.8)
- added REF**: Spacer, mylibrary:Spacer, F.Cu at (252.4, 142.5)
- added REF**: Spacer, mylibrary:Spacer, F.Cu at (288.5, 159.5)
- added REF**: Spacer, mylibrary:Spacer, F.Cu at (248.3, 267.1)
- added REF**: Spacer, mylibrary:Spacer, F.Cu at (195.3, 142.5)
- added REF**: Spacer, mylibrary:Spacer, F.Cu at (258.4, 162.1)
- added REF**: Spacer, mylibrary:Spacer, F.Cu at (162.5, 279.0)
- added REF**: Spacer, mylibrary:Spacer, F.Cu at (159.2, 162.1)
- added REF**: Spacer, mylibrary:Spacer, F.Cu at (300.0, 271.8)
- added REF**: Spacer, mylibrary:Spacer, F.Cu at (317.1, 214.1)

Commit message: トッププレート
Parts:
- added REF**: Spacer, mylibrary:Spacer, F.Cu at (159.2, -132.9)
- added REF**: Spacer, mylibrary:Spacer, F.Cu at (162.5, -21.0)
- added REF**: Spacer, mylibrary:Spacer, F.Cu at (159.2, -137.9)
- added REF**: Spacer, mylibrary:Spacer, F.Cu at (300.0, -28.2)
- added REF**: Spacer, mylibrary:Spacer, F.Cu at (317.1, -85.9)
- added REF**: Spacer, mylibrary:Spacer, F.Cu at (156.0, -82.6)
- added REF**: Spacer, mylibrary:Spacer, F.Cu at (317.1, -45.2)
- added REF**: Spacer, mylibrary:Spacer, F.Cu at (317.1, -124.2)
- added REF**: Spacer, mylibrary:Spacer, F.Cu at (252.4, -157.5)
- added REF**: Spacer, mylibrary:Spacer, F.Cu at (240.7, -94.8)
- added REF**: Spacer, mylibrary:Spacer, F.Cu at (303.5, -157.5)
- added REF**: Spacer, mylibrary:Spacer, F.Cu at (258.4, -132.9)
- added REF**: Spacer, mylibrary:Spacer, F.Cu at (248.3, -32.9)
- added REF**: Spacer, mylibrary:Spacer, F.Cu at (303.5, -137.9)
- added REF**: Spacer, mylibrary:Spacer, F.Cu at (303.5, -132.9)
- added REF**: Spacer, mylibrary:Spacer, F.Cu at (195.3, -157.5)
- added REF**: Spacer, mylibrary:Spacer, F.Cu at (258.4, -137.9)
Other:
- board size 316.7 x 290.8 mm -> 316.7 x 440.8 mm

Commit message: 左手導線
Parts:
- removed the REF** at (258.4, 162.1)
- removed the REF** at (128.3, -7.53)
- removed the REF** at (4.38, 13.8)
- removed the REF** at (4.38, 18.8)
- added REF**: Spacer, mylibrary:Spacer, F.Cu at (12.8, 13.8)
- added REF**: Spacer, mylibrary:Spacer, F.Cu at (12.8, 18.8)
- moved D1002 132.5 mm to (12.1, 29.8), turned to 180 degrees
- moved C1 131.9 mm to (123.8, 16.7)
- moved D1001 125.0 mm to (12.1, 27.3), turned to 180 degrees
- moved D1000 118.8 mm to (12.1, 24.8), turned to 180 degrees
- moved DD2 84.6 mm to (23.5, 1.27)
- moved SW1002 76.5 mm to (9.68, 20.5)
- moved DD1 66.9 mm to (23.5, -2.54)
- moved SW1000 57.4 mm to (9.68, 5.08)
- moved SW1001 48.6 mm to (9.68, 12.7)
- moved R1 35.0 mm to (23.5, -5.71), turned to 0 degrees
- moved D5 28.7 mm to (102.1, 15.2)
- moved D4 22.6 mm to (96.2, 11.9)
- moved REF** 20.3 mm to (238.1, -137.9)
- moved REF** 20.3 mm to (238.1, 12.1)
- moved D1 19.9 mm to (33.3, 9.53)
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Connections:
- BPM1 pad 10: col4 -> col2
- BPM1 pad 11: col5 -> col3
- BPM1 pad 16: row5 -> row0
- BPM1 pad 17: row4 -> row1
- BPM1 pad 18: row3 -> row2
- BPM1 pad 19: row2 -> row3
- BPM1 pad 20: row1 -> row4
- BPM1 pad 21: row0 -> row5
- BPM1 pad 6: col0 -> col5
- BPM1 pad 7: col1 -> col4
- BPM1 pad 8: col2 -> col0
- BPM1 pad 9: col3 -> col1
Routing:
- net col1: track 0.00 -> 320.7 mm
- net col0: track 0.00 -> 312.4 mm
- net col2: track 0.00 -> 309.7 mm
- net row5: track 0.00 -> 241.9 mm
- net row4: track 0.00 -> 219.9 mm
- net row3: track 0.00 -> 206.9 mm
- net row2: track 0.00 -> 186.6 mm
- net col5: track 0.00 -> 148.8 mm
- net row1: track 0.00 -> 145.4 mm
- net bat0: track 0.00 -> 144.7 mm
- net col4: track 0.00 -> 132.6 mm
- net rowsys0: track 0.00 -> 111.5 mm
- net row0: track 0.00 -> 101.2 mm
- net col3: track 0.00 -> 100.4 mm
- net led0: track 0.00 -> 69.0 mm
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Other:
- board size 316.7 x 440.8 mm -> 319.1 x 440.8 mm

Commit message: 配線できた
Parts:
- moved DD2 1.91 mm to (21.6, 1.27)
- moved D0 1.90 mm to (29.2, 4.45)
Routing:
- net gnd0: track 0.00 -> 17.8 mm
- net Net-(DD2-Pad2): track 3.33 -> 5.03 mm
- net Net-(DD1-Pad1): track 21.3 -> 20.1 mm
- net row0: track 101.2 -> 102.0 mm
- net Net-(D0-Pad2): track 11.0 -> 10.3 mm
Changed lines of the file:
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@@
     (thickness 1.6)
     (drawings 332)
-    (tracks 986)
+    (tracks 992)
     (zones 0)
     (modules 241)
@@
   )
   (setup
-    (last_trace_width 0.5)
+    (last_trace_width 0.25)
     (user_trace_width 0.5)
     (trace_clearance 0.2)
@@
   )
   (module Diode_THT:D_DO-41_SOD81_P7.62mm_Horizontal (layer F.Cu)
-    (at 23.495 1.27)
+    (at 21.59 1.27)
     (descr "Diode, DO-41_SOD81 series, Axial, Horizontal, pin pitch=7.62mm, , length*diameter=5.2*2.7mm^2, , http://www.diodes.com/_files/packages/DO-41%20(Plastic).pdf")
     (tags "Diode DO-41_SOD81 series Axial Horizontal pin pitch 7.62mm  length 5.2mm diameter 2.7mm")
@@
   )
   (module Diode_THT:D_DO-35_SOD27_P7.62mm_Horizontal (layer F.Cu)
-    (at 31.115 4.445 180)
+    (at 29.21 4.445 180)
     (descr "Diode, DO-35_SOD27 series, Axial, Horizontal, pin pitch=7.62mm, , length*diameter=4*2mm^2, , http://www.diodes.com/_files/packages/DO-35.pdf")
     (tags "Diode DO-35_SOD27 series Axial Horizontal pin pitch 7.62mm  length 4mm diameter 2mm")
@@
   (segment (start 97.710401 -4.365001) (end 95.326499 -4.365001) (width 0.25) (layer F.Cu) (net 17))
   (segment (start 100.965 -7.6196) (end 97.710401 -4.365001) (width 0.25) (layer F.Cu) (net 17))
-  (segment (start 33.3375 6.6675) (end 31.115 4.445) (width 0.25) (layer F.Cu) (net 17))
-  (segment (start 33.3375 9.525) (end 33.3375 6.6675) (width 0.25) (layer F.Cu) (net 17))
+  (segment (start 29.21 5.3975) (end 33.3375 9.525) (width 0.25) (layer F.Cu) (net 17))
+  (segment (start 29.21 4.445) (end 29.21 5.3975) (width 0.25) (layer F.Cu) (net 17))
   (segment (start 35.3025 3.87) (end 40.9575 9.525) (width 0.25) (layer B.Cu) (net 19))
   (segment (start 35.3025 -2.54) (end 35.3025 3.87) (width 0.25) (layer B.Cu) (net 19))
@@
   (segment (start 208.975 66.675) (end 213.36 66.675) (width 0.25) (layer B.Cu) (net 52))
   (segment (start 201.99 73.66) (end 208.975 66.675) (width 0.25) (layer B.Cu) (net 52))
+  (segment (start 121.506401 -1.173073) (end 121.506401 4.858999) (width 0.5) (layer F.Cu) (net 53))
+  (segment (start 121.506401 4.858999) (end 118.745 7.6204) (width 0.5) (layer F.Cu) (net 53))
+  (segment (start 119.652499 -3.026975) (end 121.506401 -1.173073) (width 0.5) (layer F.Cu) (net 53))
+  (segment (start 119.652499 -5.987099) (end 119.652499 -3.026975) (width 0.5) (layer F.Cu) (net 53))
+  (segment (start 121.285 -7.6196) (end 119.652499 -5.987099) (width 0.5) (layer F.Cu) (net 53))
   (segment (start 12.065 24.765) (end 12.065 29.845) (width 0.25) (layer B.Cu) (net 56))
+  (segment (start 16.637 20.193) (end 12.065 24.765) (width 0.25) (layer F.Cu) (net 56))
   (segment (start 16.637 12.411998) (end 16.637 20.193) (width 0.25) (layer F.Cu) (net 56))
   (segment (start 20.158998 8.89) (end 16.637 12.411998) (width 0.25) (layer F.Cu) (net 56))
-  (segment (start 22.225 8.89) (end 20.158998 8.89) (width 0.25) (layer F.Cu) (net 56))
-  (segment (start 16.637 20.193) (end 12.065 24.765) (width 0.25) (layer F.Cu) (net 56))
-  (segment (start 28.730001 2.384999) (end 22.225 8.89) (width 0.25) (layer F.Cu) (net 56))
-  (segment (start 28.730001 -4.847003) (end 28.730001 2.384999) (width 0.25) (layer F.Cu) (net 56))
-  (segment (start 31.938019 -8.055021) (end 28.730001 -4.847003) (width 0.25) (layer F.Cu) (net 56))
+  (segment (start 27.305 3.81) (end 22.225 8.89) (width 0.25) (layer F.Cu) (net 56))
   (segment (start 92.274579 -8.055021) (end 31.938019 -8.055021) (width 0.25) (layer F.Cu) (net 56))
+  (segment (start 27.305 -3.422002) (end 27.305 3.81) (width 0.25) (layer F.Cu) (net 56))
   (segment (start 92.71 -7.6196) (end 92.274579 -8.055021) (width 0.25) (layer F.Cu) (net 56))
+  (segment (start 31.938019 -8.055021) (end 27.305 -3.422002) (width 0.25) (layer F.Cu) (net 56))
+  (segment (start 22.225 8.89) (end 20.158998 8.89) (width 0.25) (layer F.Cu) (net 56))
   (segment (start 95.885 -7.6196) (end 92.71 -7.6196) (width 0.25) (layer F.Cu) (net 56))
   (segment (start 97.337999 -6.532599) (end 98.425 -7.6196) (width 0.25) (layer F.Cu) (net 57))
@@
   (segment (start 159.385 7.62) (end 159.385 9.525) (width 0.5) (layer F.Cu) (net 79))
   (segment (start 16.2525 11.7475) (end 16.2525 11.0525) (width 0.25) (layer B.Cu) (net 80))
-  (segment (start 16.2525 11.6875) (end 23.495 4.445) (width 0.25) (layer B.Cu) (net 80))
   (segment (start 16.2525 11.7475) (end 16.2525 11.6875) (width 0.25) (layer B.Cu) (net 80))
+  (segment (start 16.2525 9.7825) (end 21.59 4.445) (width 0.25) (layer B.Cu) (net 80))
+  (segment (start 16.2525 11.7475) (end 16.2525 9.7825) (width 0.25) (layer B.Cu) (net 80))
   (segment (start 8.95 104.775) (end 13.3347 104.775) (width 0.25) (layer B.Cu) (net 81))
   (segment (start 1.965 111.76) (end 8.95 104.775) (width 0.25) (layer B.Cu) (net 81))
@@
   (segment (start 35.605001 -7.030001) (end 65.388501 -7.030001) (width 0.5) (layer F.Cu) (net 133))
   (segment (start 31.115 -2.54) (end 35.605001 -7.030001) (width 0.5) (layer F.Cu) (net 133))
-  (segment (start 14.129 1.27) (end 23.495 1.27) (width 0.5) (layer F.Cu) (net 134))
   (segment (start 8.414 -4.445) (end 14.129 1.27) (width 0.5) (layer F.Cu) (net 134))
-  (segment (start 23.495 1.27) (end 23.495 -2.54) (width 0.5) (layer F.Cu) (net 134))
-  (segment (start 31.115 0.635) (end 31.325 0.635) (width 0.5) (layer F.Cu) (net 135))
+  (segment (start 14.129 1.27) (end 21.59 1.27) (width 0.5) (layer F.Cu) (net 134))
+  (segment (start 21.59 -0.635) (end 23.495 -2.54) (width 0.5) (layer F.Cu) (net 134))
+  (segment (start 21.59 1.27) (end 21.59 -0.635) (width 0.5) (layer F.Cu) (net 134))
   (segment (start 31.96 1.27) (end 33.57 2.88) (width 0.5) (layer F.Cu) (net 135))
-  (segment (start 31.115 1.27) (end 31.96 1.27) (width 0.5) (layer F.Cu) (net 135))
+  (segment (start 29.21 1.27) (end 31.96 1.27) (width 0.5) (layer F.Cu) (net 135))
   (segment (start 258.83 2.29) (end 266.7 10.16) (width 0.5) (layer F.Cu) (net 136))
   (segment (start 251.76 2.29) (end 258.83 2.29) (width 0.5) (layer F.Cu) (net 136))

Commit message: 左手穴あけ
Parts:
- removed the REF** at (307.2, 61.9)
- added REF**: Spacer, mylibrary:Spacer, F.Cu at (124.9, 67.4)
- added REF**: Spacer, mylibrary:Spacer, F.Cu at (52.4, -7.53)
- added REF**: Spacer, mylibrary:Spacer, F.Cu at (90.8, -7.53)
- added REF**: Spacer, mylibrary:Spacer, F.Cu at (126.6, 12.1)
- added REF**: Spacer, mylibrary:Spacer, F.Cu at (126.6, 17.1)
- added REF**: Stabilizer, mylibrary:Stabilizer, F.Cu at (307.2, 61.9)
- added REF**: Spacer, mylibrary:Spacer, F.Cu at (90.8, 17.1)
- added REF**: Spacer, mylibrary:Spacer, F.Cu at (71.7, 12.1)
- added REF**: Spacer, mylibrary:Spacer, F.Cu at (64.1, 55.2)
- added REF**: Spacer, mylibrary:Spacer, F.Cu at (71.8, 117.1)
- added REF**: Spacer, mylibrary:Spacer, F.Cu at (2.00, 104.8)
- added REF**: Spacer, mylibrary:Spacer, F.Cu at (2.00, 55.2)
- moved REF** 10.9 mm to (2.00, 17.1)
- moved REF** 10.9 mm to (2.00, 12.1)
- moved D13 10.8 mm to (98.4, 22.9), turned to 180 degrees
- moved D12 8.89 mm to (74.4, 9.53)
- moved D3 8.89 mm to (85.1, 9.53)
- moved SW1001 7.85 mm to (11.6, 20.3)
- moved SW1002 7.85 mm to (11.6, 28.1)
- moved SW1000 7.85 mm to (11.6, 12.7)
- moved D1000 6.98 mm to (12.1, 31.8)
- moved D1001 6.98 mm to (12.1, 34.3)
- moved D1002 6.98 mm to (12.1, 36.8)
- moved D20 5.29 mm to (12.1, 39.4), turned to 180 degrees
- moved C1 1.82 mm to (122.8, 15.2)
- moved U2 0.59 mm to (13.6, 2.29)
- moved REF** 0.30 mm to (238.4, -137.9)
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Routing:
- net col2: track 309.7 -> 331.7 mm
- net rowsys0: track 111.5 -> 123.7 mm
- net Net-(D3-Pad2): track 16.5 -> 25.6 mm
- net Net-(D12-Pad2): track 21.6 -> 30.5 mm
- net col1: track 320.7 -> 327.7 mm
- net col0: track 312.4 -> 305.6 mm
- net led0: track 69.0 -> 73.1 mm
- net bat0: track 144.7 -> 148.7 mm
- net Net-(D20-Pad2): track 14.3 -> 10.5 mm
- net row2: track 186.6 -> 183.1 mm
- net Net-(DD1-Pad2): track 48.4 -> 51.0 mm
- net col3: track 100.4 -> 99.4 mm
- net row1: track 145.4 -> 146.2 mm
- net row0: track 102.0 -> 102.5 mm

Commit message: 整理
Parts:
- removed the REF** at (2.00, -7.53)
- removed the REF** at (303.5, -157.5)
- removed the REF** at (303.5, -7.53)
- added REF**: Spacer, mylibrary:Spacer, F.Cu at (126.6, 162.1)
- added REF**: Spacer, mylibrary:Spacer, F.Cu at (124.9, 217.4)
- added REF**: Spacer, mylibrary:Spacer, F.Cu at (90.8, 142.5)
- added REF**: Spacer, mylibrary:Spacer, F.Cu at (52.4, 142.5)
- added REF**: Spacer, mylibrary:Spacer, F.Cu at (2.00, 205.2)
- added REF**: Spacer, mylibrary:Spacer, F.Cu at (2.00, 254.8)
- added REF**: Spacer, mylibrary:Spacer, F.Cu at (19.1, 267.1)
- added REF**: Spacer, mylibrary:Spacer, F.Cu at (71.8, 267.1)
- added REF**: Spacer, mylibrary:Spacer, F.Cu at (118.5, 279.0)
- added REF**: Spacer, mylibrary:Spacer, F.Cu at (64.1, 205.2)
- moved SW1002 30.1 mm to (10.8, -1.91), turned to 270 degrees
- moved LED2 21.7 mm to (302.9, -1.91), turned to 270 degrees
- moved REF** 19.0 mm to (271.5, -157.5)
- moved REF** 19.0 mm to (271.5, -7.53)
- moved LED1 16.7 mm to (2.54, -1.91), turned to 270 degrees
- moved SW1001 13.4 mm to (10.8, 6.99), turned to 270 degrees
- moved SW1003 7.73 mm to (299.1, -1.91), turned to 270 degrees
- moved SW1004 6.48 mm to (299.1, 6.99), turned to 270 degrees
- moved SW1005 5.24 mm to (299.1, 15.9), turned to 270 degrees
- moved SW1000 3.27 mm to (10.8, 15.9), turned to 270 degrees
- moved SWITCH0 2.81 mm to (6.35, -6.35)
- moved SWITCH1 2.69 mm to (299.1, -6.35)
Routing:
- net col2: track 331.7 -> 300.5 mm
- net Net-(LED2-Pad2): track 13.5 -> 43.7 mm
- net Net-(D1002-Pad2): track 16.1 -> 40.8 mm
- net col1: track 327.7 -> 309.8 mm
- net Net-(LED1-Pad2): track 7.51 -> 23.6 mm
- net Net-(D1000-Pad2): track 26.5 -> 16.6 mm
- net Net-(D1001-Pad2): track 21.4 -> 29.0 mm
- net Net-(D1004-Pad2): track 21.8 -> 15.8 mm
- net Net-(D1005-Pad2): track 19.3 -> 13.4 mm
- net col13: track 353.5 -> 359.1 mm
- net Net-(D1003-Pad2): track 26.5 -> 22.3 mm
- net col11: track 382.6 -> 378.7 mm
- net Net-(DD1-Pad1): track 20.1 -> 24.0 mm
- net col12: track 365.6 -> 361.9 mm
- net Net-(DD3-Pad1): track 32.7 -> 35.4 mm
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Other:
- outline, holes or cut-outs redrawn

Commit message: gnd
Parts:
- added REF**: Spacer, mylibrary:Spacer, F.Cu at (16.3, 23.8)
- moved D0 36.1 mm to (40.6, 38.7)
- moved DD2 36.1 mm to (33.0, 35.6)
- moved DD1 36.1 mm to (34.9, 31.8)
- moved R1 36.1 mm to (34.9, 28.6)
- moved D1001 35.9 mm to (20.3, 69.2), turned to 270 degrees
- moved D1002 34.1 mm to (22.9, 69.2), turned to 270 degrees
- moved D1000 21.3 mm to (22.9, 50.2), turned to 270 degrees
- moved REF** 19.0 mm to (271.5, 142.5)
- moved D20 13.6 mm to (20.3, 50.2), turned to 270 degrees
- moved D15 1.73 mm to (117.8, 25.6)
Routing:
- net led0: track 73.1 -> 170.0 mm
- net Net-(DD1-Pad2): track 51.0 -> 139.3 mm
- net Net-(DD2-Pad2): track 4.78 -> 80.3 mm
- net row0: track 102.5 -> 156.8 mm
- net Net-(DD1-Pad1): track 24.0 -> 78.1 mm
- net Net-(LED1-Pad2): track 23.6 -> 76.8 mm
- net Net-(D1002-Pad2): track 40.8 -> 93.3 mm
- net Net-(D1001-Pad2): track 29.0 -> 81.3 mm
- net rowsys0: track 123.7 -> 168.6 mm
- net Net-(D0-Pad2): track 10.3 -> 53.8 mm
- net col0: track 305.0 -> 340.2 mm
- net Net-(D1000-Pad2): track 16.6 -> 50.1 mm
- net Net-(D20-Pad2): track 10.5 -> 20.3 mm
- net col5: track 148.8 -> 153.2 mm
- net row1: track 146.2 -> 144.3 mm
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
Commit message: 穴途中
Parts:
- added REF**: Spacer, mylibrary:Spacer, F.Cu at (126.6, -132.9)
- added REF**: Spacer, mylibrary:Spacer, F.Cu at (71.8, -32.9)
- added REF**: Spacer, mylibrary:Spacer, F.Cu at (118.5, -21.0)
- added REF**: Spacer, mylibrary:Spacer, F.Cu at (64.1, -94.8)
- added REF**: Spacer, mylibrary:Spacer, F.Cu at (71.7, -137.9)
- added REF**: Spacer, mylibrary:Spacer, F.Cu at (90.8, -132.9)
- added REF**: Spacer, mylibrary:Spacer, F.Cu at (124.9, -82.6)
- added REF**: Spacer, mylibrary:Spacer, F.Cu at (16.3, 173.8)
- added REF**: Spacer, mylibrary:Spacer, F.Cu at (126.6, -137.9)
- added REF**: Spacer, mylibrary:Spacer, F.Cu at (90.8, -157.5)
- added REF**: Spacer, mylibrary:Spacer, F.Cu at (52.4, -157.5)
- added REF**: Spacer, mylibrary:Spacer, F.Cu at (2.00, -137.9)
- added REF**: Spacer, mylibrary:Spacer, F.Cu at (2.00, -132.9)
- added REF**: Spacer, mylibrary:Spacer, F.Cu at (2.00, -94.8)
- added REF**: Spacer, mylibrary:Spacer, F.Cu at (2.00, -45.2)
- added REF**: Spacer, mylibrary:Spacer, F.Cu at (19.1, -32.9)
Other:
- outline, holes or cut-outs redrawn
