File: Right/Right.sch (KiCad schematic (older format))
At the start: 105 parts, among them SW1 SW_PUSH, SW10 SW_PUSH, SW100 SW_Push_Dual_R, SW101 SW_Push_Dual_R, SW102 SW_Push_Dual_R, SW11 SW_PUSH, SW12 SW_PUSH, SW13 SW_PUSH, SW14 SW_PUSH, SW15 SW_PUSH, SW16 SW_PUSH, SW17 SW_PUSH, SW18 SW_PUSH, SW19 SW_PUSH, SW2 SW_PUSH, SW20 SW_PUSH, SW200 SW_SPDT, SW21 SW_PUSH, SW22 SW_PUSH, SW23 SW_PUSH, SW24 SW_PUSH, SW25 SW_PUSH, SW26 SW_PUSH, SW27 SW_PUSH, SW28 SW_PUSH, SW29 SW_PUSH, SW3 SW_PUSH, SW30 SW_PUSH, SW31 SW_PUSH, SW32 SW_PUSH, SW33 SW_PUSH, SW34 SW_PUSH, SW35 SW_PUSH, SW36 SW_PUSH, SW37 SW_PUSH, SW38 SW_PUSH, SW39 SW_PUSH, SW4 SW_PUSH, SW40 SW_PUSH, SW41 SW_PUSH, SW42 SW_PUSH, SW43 SW_PUSH, SW44 SW_PUSH, SW45 SW_PUSH, SW5 SW_PUSH, SW6 SW_PUSH, SW7 SW_PUSH, SW8 SW_PUSH, SW9 SW_PUSH, U1 CH25-2032LF, U2 CH25-2032LF

Commit message: 小さく
Connections:
- net col0: now also BPM1.21 (PIN20); no longer BPM1.14 (PIN13), SW100.1
- net col1: now also BPM1.20 (PIN19); no longer BPM1.15 (PIN14), SW101.1
- net col2: now also BPM1.19 (PIN18); no longer BPM1.16 (PIN15), SW102.1
- net col3: now also BPM1.18 (PIN17); no longer BPM1.17 (PIN16)
- net col4: now also BPM1.17 (PIN16); no longer BPM1.18 (PIN17)
- net col5: now also BPM1.16 (PIN15), SW100.1; no longer BPM1.19 (PIN18)
- net col6: now also BPM1.15 (PIN14), SW101.1; no longer BPM1.20 (PIN19)
- net col7: now also BPM1.14 (PIN13), SW102.1; no longer BPM1.21 (PIN20)
Other:
- moved on the sheet: D100, D101, D102, SW100, SW101, SW102
Changed lines of the file:
@@
 $EndComp
 Wire Wire Line
-	5750 1200 5750 1750
+	10000 1200 10000 1750
 Connection ~ 5750 2700
 Connection ~ 6350 3000
@@
 	0    -1   -1   0
 $EndComp
-Wire Wire Line
-	8300 2400 8300 2700
 Connection ~ 8300 2700
 Connection ~ 8900 3000
@@
 	0    -1   -1   0
 $EndComp
-Wire Wire Line
-	9150 2400 9150 2700
 Connection ~ 9150 2700
 Connection ~ 9750 3000
@@
 	0    -1   -1   0
 $EndComp
-Wire Wire Line
-	10000 2400 10000 2700
 Connection ~ 10000 2700
 Wire Wire Line
@@
 Text GLabel 4000 6250 0    50   Input ~ 0
 row5
-Text GLabel 4050 1250 1    50   Input ~ 0
+Text GLabel 4050 2400 1    50   Input ~ 0
 col0
-Text GLabel 4900 1200 1    50   Input ~ 0
+Text GLabel 4900 2400 1    50   Input ~ 0
 col1
-Text GLabel 5750 1200 1    50   Input ~ 0
+Text GLabel 5750 2400 1    50   Input ~ 0
 col2
 Text GLabel 6600 2400 1    50   Input ~ 0
@@
 Text GLabel 7450 2400 1    50   Input ~ 0
 col4
-Text GLabel 8300 2400 1    50   Input ~ 0
+Text GLabel 8300 1250 1    50   Input ~ 0
 col5
-Text GLabel 9150 2400 1    50   Input ~ 0
+Text GLabel 9150 1200 1    50   Input ~ 0
 col6
-Text GLabel 10000 2400 1    50   Input ~ 0
+Text GLabel 10000 1200 1    50   Input ~ 0
 col7
 $Comp
@@
 Text GLabel 1150 1850 0    50   Input ~ 0
 row5
-Text GLabel 2550 2550 2    50   Input ~ 0
-col0
-Text GLabel 2550 2450 2    50   Input ~ 0
-col1
-Text GLabel 2550 2350 2    50   Input ~ 0
-col2
-Text GLabel 2550 2250 2    50   Input ~ 0
-col3
-Text GLabel 2550 2150 2    50   Input ~ 0
-col4
-Text GLabel 2550 2050 2    50   Input ~ 0
-col5
-Text GLabel 2550 1950 2    50   Input ~ 0
-col6
-Text GLabel 2550 1850 2    50   Input ~ 0
-col7
 $Comp
 L CH25-2032LF:CH25-2032LF U1
@@
 	1100 3900 1100 3650
 NoConn ~ 2700 3750
-NoConn ~ 4200 1950
-NoConn ~ 4600 1950
+NoConn ~ 8450 1950
+NoConn ~ 8850 1950
 $Comp
 L Device:D D100
 U 1 1 5F386B99
-P 4700 1900
-F 0 "D100" V 4746 1820 50  0000 R CNN
-F 1 "D" V 4655 1820 50  0000 R CNN
-F 2 "Diode_THT:D_DO-35_SOD27_P7.62mm_Horizontal" H 4700 1900 50  0001 C CNN
-F 3 "~" H 4700 1900 50  0001 C CNN
-	1    4700 1900
-	0    -1   -1   0
-$EndComp
-Wire Wire Line
-	4600 1750 4700 1750
-Wire Wire Line
-	4700 2050 4000 2050
-Text GLabel 4000 2050 0    50   Input ~ 0
+P 8950 1900
+F 0 "D100" V 8996 1820 50  0000 R CNN
+F 1 "D" V 8905 1820 50  0000 R CNN
+F 2 "Diode_THT:D_DO-35_SOD27_P7.62mm_Horizontal" H 8950 1900 50  0001 C CNN
+F 3 "~" H 8950 1900 50  0001 C CNN
+	1    8950 1900
+	0    -1   -1   0
+$EndComp
+Wire Wire Line
+	8850 1750 8950 1750
+Wire Wire Line
+	8950 2050 8250 2050
+Text GLabel 8250 2050 0    50   Input ~ 0
 rowsys
 Wire Wire Line
-	4700 2050 5550 2050
-Connection ~ 4700 2050
-Wire Wire Line
-	4050 1250 4050 1750
-Wire Wire Line
-	4200 1750 4050 1750
-Connection ~ 4050 1750
-Wire Wire Line
-	4050 1750 4050 2700
-Wire Wire Line
-	4900 1200 4900 1750
-NoConn ~ 5050 1950
-NoConn ~ 5450 1950
+	8950 2050 9800 2050
+Connection ~ 8950 2050
+Wire Wire Line
+	8300 1250 8300 1750
+Wire Wire Line
+	8450 1750 8300 1750
+Connection ~ 8300 1750
+Wire Wire Line
+	9150 1200 9150 1750
+NoConn ~ 9300 1950
+NoConn ~ 9700 1950
 $Comp
 L Device:D D101
 U 1 1 5F3CEA11
-P 5550 1900
-F 0 "D101" V 5596 1820 50  0000 R CNN
-F 1 "D" V 5505 1820 50  0000 R CNN
-F 2 "Diode_THT:D_DO-35_SOD27_P7.62mm_Horizontal" H 5550 1900 50  0001 C CNN
-F 3 "~" H 5550 1900 50  0001 C CNN
-	1    5550 1900
-	0    -1   -1   0
-$EndComp
-Wire Wire Line
-	5450 1750 5550 1750
-Wire Wire Line
-	5050 1750 4900 1750
-Connection ~ 5550 2050
-Connection ~ 4900 1750
-Wire Wire Line
-	4900 1750 4900 2700
-NoConn ~ 5900 1950
-NoConn ~ 6300 1950
+P 9800 1900
+F 0 "D101" V 9846 1820 50  0000 R CNN
+F 1 "D" V 9755 1820 50  0000 R CNN
+F 2 "Diode_THT:D_DO-35_SOD27_P7.62mm_Horizontal" H 9800 1900 50  0001 C CNN
+F 3 "~" H 9800 1900 50  0001 C CNN
+	1    9800 1900
+	0    -1   -1   0
+$EndComp
+Wire Wire Line
+	9700 1750 9800 1750
+Wire Wire Line
+	9300 1750 9150 1750
+Connection ~ 9800 2050
+Connection ~ 9150 1750
+NoConn ~ 10150 1950
+NoConn ~ 10550 1950
 $Comp
 L Device:D D102
 U 1 1 5F3D4407
-P 6400 1900
-F 0 "D102" V 6446 1820 50  0000 R CNN
-F 1 "D" V 6355 1820 50  0000 R CNN
-F 2 "Diode_THT:D_DO-35_SOD27_P7.62mm_Horizontal" H 6400 1900 50  0001 C CNN
-F 3 "~" H 6400 1900 50  0001 C CNN
-	1    6400 1900
-	0    -1   -1   0
-$EndComp
-Wire Wire Line
-	6300 1750 6400 1750
-Wire Wire Line
-	5900 1750 5750 1750
-Connection ~ 5750 1750
-Wire Wire Line
-	5750 1750 5750 2700
-Wire Wire Line
-	5550 2050 6400 2050
+P 10650 1900
+F 0 "D102" V 10696 1820 50  0000 R CNN
+F 1 "D" V 10605 1820 50  0000 R CNN
+F 2 "Diode_THT:D_DO-35_SOD27_P7.62mm_Horizontal" H 10650 1900 50  0001 C CNN
+F 3 "~" H 10650 1900 50  0001 C CNN
+	1    10650 1900
+	0    -1   -1   0
+$EndComp
+Wire Wire Line
+	10550 1750 10650 1750
+Wire Wire Line
+	10150 1750 10000 1750
+Connection ~ 10000 1750
+Wire Wire Line
+	9800 2050 10650 2050
 Text GLabel 1150 2550 0    50   Input ~ 0
 rowsys
@@
 L My_Library:SW_Push_Dual_R SW102
 U 1 1 5F449060
-P 6100 1750
-F 0 "SW102" H 6100 2035 50  0000 C CNN
-F 1 "SW_Push_Dual_R" H 6100 1944 50  0000 C CNN
-F 2 "Button_Switch_THT:SW_TH_Tactile_Omron_B3F-10xx" H 6100 1950 50  0001 C CNN
-F 3 "" H 6100 1950 50  0001 C CNN
-	1    6100 1750
+P 10350 1750
+F 0 "SW102" H 10350 2035 50  0000 C CNN
+F 1 "SW_Push_Dual_R" H 10350 1944 50  0000 C CNN
+F 2 "Button_Switch_THT:SW_TH_Tactile_Omron_B3F-10xx" H 10350 1950 50  0001 C CNN
+F 3 "" H 10350 1950 50  0001 C CNN
+	1    10350 1750
 	1    0    0    -1
 $EndComp
@@
 L My_Library:SW_Push_Dual_R SW101
 U 1 1 5F44E520
-P 5250 1750
-F 0 "SW101" H 5250 2035 50  0000 C CNN
-F 1 "SW_Push_Dual_R" H 5250 1944 50  0000 C CNN
-F 2 "Button_Switch_THT:SW_TH_Tactile_Omron_B3F-10xx" H 5250 1950 50  0001 C CNN
-F 3 "" H 5250 1950 50  0001 C CNN
-	1    5250 1750
+P 9500 1750
+F 0 "SW101" H 9500 2035 50  0000 C CNN
+F 1 "SW_Push_Dual_R" H 9500 1944 50  0000 C CNN
+F 2 "Button_Switch_THT:SW_TH_Tactile_Omron_B3F-10xx" H 9500 1950 50  0001 C CNN
+F 3 "" H 9500 1950 50  0001 C CNN
+	1    9500 1750
 	1    0    0    -1
 $EndComp
@@
 L My_Library:SW_Push_Dual_R SW100
 U 1 1 5F44F80F
-P 4400 1750
-F 0 "SW100" H 4400 2035 50  0000 C CNN
-F 1 "SW_Push_Dual_R" H 4400 1944 50  0000 C CNN
-F 2 "Button_Switch_THT:SW_TH_Tactile_Omron_B3F-10xx" H 4400 1950 50  0001 C CNN
-F 3 "" H 4400 1950 50  0001 C CNN
-	1    4400 1750
-	1    0    0    -1
-$EndComp
+P 8650 1750
+F 0 "SW100" H 8650 2035 50  0000 C CNN
+F 1 "SW_Push_Dual_R" H 8650 1944 50  0000 C CNN
+F 2 "Button_Switch_THT:SW_TH_Tactile_Omron_B3F-10xx" H 8650 1950 50  0001 C CNN
+F 3 "" H 8650 1950 50  0001 C CNN
+	1    8650 1750
+	1    0    0    -1
+$EndComp
+Wire Wire Line
+	5750 2400 5750 2700
+Wire Wire Line
+	4900 2400 4900 2700
+Wire Wire Line
+	4050 2400 4050 2700
+Wire Wire Line
+	8300 1750 8300 2700
+Wire Wire Line
+	9150 1750 9150 2700
+Wire Wire Line
+	10000 1750 10000 2700
+Text GLabel 2550 2550 2    50   Input ~ 0
+col7
+Text GLabel 2550 2450 2    50   Input ~ 0
+col6
+Text GLabel 2550 2350 2    50   Input ~ 0
+col5
+Text GLabel 2550 2250 2    50   Input ~ 0
+col4
+Text GLabel 2550 2150 2    50   Input ~ 0
+col3
+Text GLabel 2550 2050 2    50   Input ~ 0
+col2
+Text GLabel 2550 1950 2    50   Input ~ 0
+col1
+Text GLabel 2550 1850 2    50   Input ~ 0
+col0
 $EndSCHEMATC

Commit message: 位置調整
Parts:
- BPM1: footprint mylibrary:BLEMicroPro_reversed -> mylibrary:BLEMicroPro
Connections:
- net col0: now also BPM1.6 (PIN5); no longer BPM1.21 (PIN20)
- net col1: now also BPM1.7 (PIN6); no longer BPM1.20 (PIN19)
- net col2: now also BPM1.8 (PIN7); no longer BPM1.19 (PIN18)
- net col3: now also BPM1.9 (PIN8); no longer BPM1.18 (PIN17)
- net col4: now also BPM1.10 (PIN9); no longer BPM1.17 (PIN16)
- net col5: now also BPM1.11 (PIN10); no longer BPM1.16 (PIN15)
- net col6: now also BPM1.12 (PIN11); no longer BPM1.15 (PIN14)
- net col7: now also BPM1.13 (PIN12); no longer BPM1.14 (PIN13)
- net led: now also BPM1.15 (PIN14); no longer BPM1.12 (PIN11)
- net row0: now also BPM1.16 (PIN15); no longer BPM1.11 (PIN10)
- net row1: now also BPM1.17 (PIN16); no longer BPM1.10 (PIN9)
- net row2: now also BPM1.18 (PIN17); no longer BPM1.9 (PIN8)
- net row3: now also BPM1.19 (PIN18); no longer BPM1.8 (PIN7)
- net row4: now also BPM1.20 (PIN19); no longer BPM1.7 (PIN6)
- net row5: now also BPM1.21 (PIN20); no longer BPM1.6 (PIN5)
- net rowsys: now also BPM1.14 (PIN13); no longer BPM1.13 (PIN12)
Changed lines of the file:
@@
 F 0 "BPM1" H 1850 3337 60  0000 C CNN
 F 1 "BleProMicro" H 1850 3231 60  0000 C CNN
-F 2 "mylibrary:BLEMicroPro_reversed" H 1950 1150 60  0001 C CNN
+F 2 "mylibrary:BLEMicroPro" H 1950 1150 60  0001 C CNN
 F 3 "" H 1950 1150 60  0000 C CNN
 	1    1850 2200
 	1    0    0    -1
 $EndComp
-Text GLabel 1150 2350 0    50   Input ~ 0
+Text GLabel 2550 2350 2    50   Input ~ 0
 row0
-Text GLabel 1150 2250 0    50   Input ~ 0
+Text GLabel 2550 2250 2    50   Input ~ 0
 row1
-Text GLabel 1150 2150 0    50   Input ~ 0
+Text GLabel 2550 2150 2    50   Input ~ 0
 row2
-Text GLabel 1150 2050 0    50   Input ~ 0
+Text GLabel 2550 2050 2    50   Input ~ 0
 row3
-Text GLabel 1150 1950 0    50   Input ~ 0
+Text GLabel 2550 1950 2    50   Input ~ 0
 row4
-Text GLabel 1150 1850 0    50   Input ~ 0
+Text GLabel 2550 1850 2    50   Input ~ 0
 row5
 $Comp
@@
 Text GLabel 1350 5150 0    50   Input ~ 0
 led
-Text GLabel 1150 2450 0    50   Input ~ 0
+Text GLabel 2550 2450 2    50   Input ~ 0
 led
 Wire Wire Line
@@
 Wire Wire Line
 	9800 2050 10650 2050
-Text GLabel 1150 2550 0    50   Input ~ 0
+Text GLabel 2550 2550 2    50   Input ~ 0
 rowsys
 $Comp
@@
 Wire Wire Line
 	10000 1750 10000 2700
-Text GLabel 2550 2550 2    50   Input ~ 0
+Text GLabel 1150 1850 0    50   Input ~ 0
+col0
+Text GLabel 1150 1950 0    50   Input ~ 0
+col1
+Text GLabel 1150 2050 0    50   Input ~ 0
+col2
+Text GLabel 1150 2150 0    50   Input ~ 0
+col3
+Text GLabel 1150 2250 0    50   Input ~ 0
+col4
+Text GLabel 1150 2350 0    50   Input ~ 0
+col5
+Text GLabel 1150 2450 0    50   Input ~ 0
+col6
+Text GLabel 1150 2550 0    50   Input ~ 0
 col7
-Text GLabel 2550 2450 2    50   Input ~ 0
-col6
-Text GLabel 2550 2350 2    50   Input ~ 0
-col5
-Text GLabel 2550 2250 2    50   Input ~ 0
-col4
-Text GLabel 2550 2150 2    50   Input ~ 0
-col3
-Text GLabel 2550 2050 2    50   Input ~ 0
-col2
-Text GLabel 2550 1950 2    50   Input ~ 0
-col1
-Text GLabel 2550 1850 2    50   Input ~ 0
-col0
 $EndSCHEMATC

Commit message: 全体にした
Parts:
- removed D36, D37, D38, D39, D40, D41, D42, D43, D44, D45: D, Diode_THT:D_DO-35_SOD27_P7.62mm_Horizontal, symbol Device:D
- removed SW36, SW37, SW38, SW39, SW40, SW41, SW42, SW43, SW44, SW45: SW_PUSH, keyswitches:Kailh_socket_MX, symbol kbd:SW_PUSH
- added BPM2: BleProMicro, mylibrary:BLEMicroPro, symbol My_Library:BleProMicro
- added C2: C, Capacitor_THT:C_Disc_D5.1mm_W3.2mm_P5.00mm, symbol Device:C
- added D100, D1003, D1004, D1005, D101, D102, D103, D104, D105, D106, D110, D111, D112, D113, D114, D115, D116, D60, D61, D62, D63, D64, D65, D66, D70, D71, D72, D73, D74, D75, D76, D77, D80, D81, D82, D83, D84, D85, D86, D87, D90, D91, D92, D93, D94, D95, D96: D, Diode_THT:D_DO-35_SOD27_P7.62mm_Horizontal, symbol Device:D
- added DD3, DD4: D, Diode_THT:D_DO-41_SOD81_P7.62mm_Horizontal, symbol Device:D
- added LED2: LED, LED_THT:LED_D3.0mm, symbol Device:LED
- added R2: R, Resistor_THT:R_Axial_DIN0204_L3.6mm_D1.6mm_P7.62mm_Horizontal, symbol Device:R
- added SW100, SW101, SW102, SW103, SW104, SW105, SW106, SW110, SW111, SW112, SW113, SW114, SW115, SW116, SW60, SW61, SW62, SW63, SW64, SW65, SW66, SW70, SW71, SW72, SW73, SW74, SW75, SW76, SW77, SW80, SW81, SW82, SW83, SW84, SW85, SW86, SW87, SW90, SW91, SW92, SW93, SW94, SW95, SW96: SW_PUSH, keyswitches:Kailh_socket_MX, symbol kbd:SW_PUSH
- added SW1003, SW1004, SW1005: SW_Push_Dual_R, Button_Switch_THT:SW_TH_Tactile_Omron_B3F-10xx, symbol My_Library:SW_Push_Dual_R
- added SWITCH1: SW_SPDT, mylibrary:2MS1-T1-B4-VS2-Q-E-S, symbol Switch:SW_SPDT
- added U3, U4: CH25-2032LF, CH25-2032LF:CH252032LF, symbol CH25-2032LF:CH25-2032LF
- renumbered D1 to D0, D7 to D1, D2 to D10, D100 to D1000, D101 to D1001, D102 to D1002, D8 to D11, D14 to D12, D20 to D13, D26 to D14, D31 to D15, D13 to D2, D3 to D20, D9 to D21, D15 to D22, D21 to D23, D27 to D24, D32 to D25, D19 to D3, D4 to D30, D10 to D31, D16 to D32, D22 to D33, D28 to D34, D33 to D35, D25 to D4, D5 to D40, D11 to D41, D17 to D42, D23 to D43, D29 to D44, D34 to D45, D30 to D5, D6 to D50, D12 to D51, D18 to D52, D24 to D53, D35 to D54, D200 to DD1, D201 to DD2, SW1 to SW0, SW7 to SW1, SW2 to SW10, SW100 to SW1000, SW101 to SW1001, SW102 to SW1002, SW8 to SW11, SW14 to SW12, SW20 to SW13, SW26 to SW14, SW31 to SW15, SW13 to SW2, SW3 to SW20, SW9 to SW21, SW15 to SW22, SW21 to SW23, SW27 to SW24, SW32 to SW25, SW19 to SW3, SW4 to SW30, SW10 to SW31, SW16 to SW32, SW22 to SW33, SW28 to SW34, SW33 to SW35, SW25 to SW4, SW5 to SW40, SW11 to SW41, SW17 to SW42, SW23 to SW43, SW29 to SW44, SW34 to SW45, SW30 to SW5, SW6 to SW50, SW12 to SW51, SW18 to SW52, SW24 to SW53, SW35 to SW54, SW200 to SWITCH0
Connections:
- net col0: now also SW1000.1
- net col1: now also SW1001.1
- net col2: now also SW1002.1
- net col3: no longer SW53.1
- net col4: now also SW53.1
- net col5: no longer SW1000.1
- net col6: now also BPM2.6 (PIN5), SW100.1, SW110.1, SW60.1, SW70.1, SW80.1, SW90.1; no longer BPM1.12 (PIN11), SW1001.1
- net col7: now also BPM2.7 (PIN6), SW101.1, SW111.1, SW61.1, SW71.1, SW81.1, SW91.1; no longer BPM1.13 (PIN12), SW1002.1
- net bat renamed bat0
- net gnd renamed gnd0
- net led renamed led0
- net rowsys renamed rowsys0
- new net: D61.2 (A), SW61.2
- new net: D60.2 (A), SW60.2
- new net: D62.2 (A), SW62.2
- new net: D63.2 (A), SW63.2
- new net: D65.2 (A), SW65.2
- new net: D64.2 (A), SW64.2
- new net: D66.2 (A), SW66.2
- new net: D71.2 (A), SW71.2
- new net: D70.2 (A), SW70.2
- new net: D72.2 (A), SW72.2
- new net: D73.2 (A), SW73.2
- new net: D75.2 (A), SW75.2
- new net: D74.2 (A), SW74.2
- new net: D76.2 (A), SW76.2
- new net: D77.2 (A), SW77.2
- new net: D81.2 (A), SW81.2
- new net: D80.2 (A), SW80.2
- new net: D82.2 (A), SW82.2
- new net: D83.2 (A), SW83.2
- new net: D85.2 (A), SW85.2
- new net: D84.2 (A), SW84.2
- new net: D86.2 (A), SW86.2
- new net: D87.2 (A), SW87.2
- new net: D91.2 (A), SW91.2
- new net: D90.2 (A), SW90.2
- new net: D92.2 (A), SW92.2
- new net: D93.2 (A), SW93.2
- new net: D95.2 (A), SW95.2
- new net: D94.2 (A), SW94.2
- new net: D96.2 (A), SW96.2
- new net: D101.2 (A), SW101.2
- new net: D100.2 (A), SW100.2
- new net: D102.2 (A), SW102.2
- new net: D103.2 (A), SW103.2
- new net: D105.2 (A), SW105.2
- new net: D104.2 (A), SW104.2
- new net: D106.2 (A), SW106.2
- new net: D111.2 (A), SW111.2
- new net: D110.2 (A), SW110.2
- new net: D112.2 (A), SW112.2
- new net: D113.2 (A), SW113.2
- new net: D114.2 (A), SW114.2
- new net: D115.2 (A), SW115.2
- new net: DD3.2 (A), U3.2 (+)
- new net: DD3.1 (K), DD4.1 (K), SWITCH1.2 (B)
- new net: DD4.2 (A), U4.2 (+)
- new net: LED2.2 (A), R2.1
- new net: D116.2 (A), SW116.2
- new net: D1003.2 (A), SW1003.3
- new net: D1004.2 (A), SW1004.3
- new net: D1005.2 (A), SW1005.3
- new net bat1: BPM2.26 (BAT), C2.1, SWITCH1.1 (A)
- new net col10: BPM2.10 (PIN9), SW104.1, SW64.1, SW74.1, SW84.1, SW94.1
- new net col11: BPM2.11 (PIN10), SW1003.1, SW105.1, SW114.1, SW65.1, SW75.1, SW85.1, SW95.1
- new net col12: BPM2.12 (PIN11), SW1004.1, SW106.1, SW115.1, SW66.1, SW76.1, SW86.1, SW96.1
- new net col13: BPM2.13 (PIN12), SW1005.1, SW116.1, SW77.1, SW87.1
- new net col8: BPM2.8 (PIN7), SW102.1, SW112.1, SW62.1, SW72.1, SW82.1, SW92.1
- new net col9: BPM2.9 (PIN8), SW103.1, SW113.1, SW63.1, SW73.1, SW83.1, SW93.1
- new net gnd1: BPM2.1 (GND), BPM2.24 (GND), BPM2.4 (GND), BPM2.5 (GND), C2.2, LED2.1 (K), U3.1 (-), U4.1 (-)
- new net led1: BPM2.15 (PIN14), R2.2
- new net row10: BPM2.20 (PIN19), D100.1 (K), D101.1 (K), D102.1 (K), D103.1 (K), D104.1 (K), D105.1 (K), D106.1 (K)
- new net row11: BPM2.21 (PIN20), D110.1 (K), D111.1 (K), D112.1 (K), D113.1 (K), D114.1 (K), D115.1 (K), D116.1 (K)
- new net row6: BPM2.16 (PIN15), D60.1 (K), D61.1 (K), D62.1 (K), D63.1 (K), D64.1 (K), D65.1 (K), D66.1 (K)
- new net row7: BPM2.17 (PIN16), D70.1 (K), D71.1 (K), D72.1 (K), D73.1 (K), D74.1 (K), D75.1 (K), D76.1 (K), D77.1 (K)
- new net row8: BPM2.18 (PIN17), D80.1 (K), D81.1 (K), D82.1 (K), D83.1 (K), D84.1 (K), D85.1 (K), D86.1 (K), D87.1 (K)
- new net row9: BPM2.19 (PIN18), D90.1 (K), D91.1 (K), D92.1 (K), D93.1 (K), D94.1 (K), D95.1 (K), D96.1 (K)
- new net rowsys1: BPM2.14 (PIN13), D1003.1 (K), D1004.1 (K), D1005.1 (K)
- no-connect marks 12 -> 26
Other:
- moved on the sheet: D1000, D1001, D1002, D53, SW1000, SW1001, SW1002, SW53

Commit message: 途中
Other:
- moved on the sheet: BPM1, BPM2, C1, C2, D0, D1, D10, D100, D1000, D1001, D1002, D1003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

Commit message: 途中
Connections:
- net col10: now also BPM2.17 (PIN16); no longer BPM2.10 (PIN9)
- net col11: now also BPM2.16 (PIN15); no longer BPM2.11 (PIN10)
- net col12: now also BPM2.15 (PIN14); no longer BPM2.12 (PIN11)
- net col13: now also BPM2.14 (PIN13); no longer BPM2.13 (PIN12)
- net col6: now also BPM2.21 (PIN20); no longer BPM2.6 (PIN5)
- net col7: now also BPM2.20 (PIN19); no longer BPM2.7 (PIN6)
- net col8: now also BPM2.19 (PIN18); no longer BPM2.8 (PIN7)
- net col9: now also BPM2.18 (PIN17); no longer BPM2.9 (PIN8)
- net led1: now also BPM2.12 (PIN11); no longer BPM2.15 (PIN14)
- net row0: now also BPM1.21 (PIN20); no longer BPM1.16 (PIN15)
- net row1: now also BPM1.20 (PIN19); no longer BPM1.17 (PIN16)
- net row10: now also BPM2.7 (PIN6); no longer BPM2.20 (PIN19)
- net row11: now also BPM2.6 (PIN5); no longer BPM2.21 (PIN20)
- net row2: now also BPM1.19 (PIN18); no longer BPM1.18 (PIN17)
- net row3: now also BPM1.18 (PIN17); no longer BPM1.19 (PIN18)
- net row4: now also BPM1.17 (PIN16); no longer BPM1.20 (PIN19)
- net row5: now also BPM1.16 (PIN15); no longer BPM1.21 (PIN20)
- net row6: now also BPM2.11 (PIN10); no longer BPM2.16 (PIN15)
- net row7: now also BPM2.10 (PIN9); no longer BPM2.17 (PIN16)
- net row8: now also BPM2.9 (PIN8); no longer BPM2.18 (PIN17)
- net row9: now also BPM2.8 (PIN7); no longer BPM2.19 (PIN18)
- net rowsys1: now also BPM2.13 (PIN12); no longer BPM2.14 (PIN13)
Other:
- moved on the sheet: BPM1, BPM2, C1, C2, D0, D1, D10, D100, D1000, D1001, D1002, D1003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

Commit message: とりあえず右手全部つながった
Connections:
- net col10: now also BPM2.16 (PIN15); no longer BPM2.17 (PIN16)
- net col11: now also BPM2.17 (PIN16); no longer BPM2.16 (PIN15)
- net col12: now also BPM2.18 (PIN17); no longer BPM2.15 (PIN14)
- net col13: now also BPM2.19 (PIN18); no longer BPM2.14 (PIN13)
- net col8: now also BPM2.14 (PIN13); no longer BPM2.19 (PIN18)
- net col9: now also BPM2.15 (PIN14); no longer BPM2.18 (PIN17)
Changed lines of the file:
@@
 Text GLabel 9950 2500 2    50   Input ~ 0
 col7
+Text GLabel 9950 3100 2    50   Input ~ 0
+col8
+Text GLabel 9950 3000 2    50   Input ~ 0
+col9
+Text GLabel 9950 2900 2    50   Input ~ 0
+col10
+Text GLabel 9950 2800 2    50   Input ~ 0
+col11
+Text GLabel 9950 2700 2    50   Input ~ 0
+col12
 Text GLabel 9950 2600 2    50   Input ~ 0
-col8
-Text GLabel 9950 2700 2    50   Input ~ 0
-col9
-Text GLabel 9950 2800 2    50   Input ~ 0
-col10
-Text GLabel 9950 2900 2    50   Input ~ 0
-col11
-Text GLabel 9950 3000 2    50   Input ~ 0
-col12
-Text GLabel 9950 3100 2    50   Input ~ 0
 col13
 $EndSCHEMATC

Commit message: 左手導線
Connections:
- net col0: now also BPM1.8 (PIN7); no longer BPM1.6 (PIN5)
- net col1: now also BPM1.9 (PIN8); no longer BPM1.7 (PIN6)
- net col2: now also BPM1.10 (PIN9); no longer BPM1.8 (PIN7)
- net col3: now also BPM1.11 (PIN10); no longer BPM1.9 (PIN8)
- net col4: now also BPM1.7 (PIN6); no longer BPM1.10 (PIN9)
- net col5: now also BPM1.6 (PIN5); no longer BPM1.11 (PIN10)
- net row0: now also BPM1.16 (PIN15); no longer BPM1.21 (PIN20)
- net row1: now also BPM1.17 (PIN16); no longer BPM1.20 (PIN19)
- net row2: now also BPM1.18 (PIN17); no longer BPM1.19 (PIN18)
- net row3: now also BPM1.19 (PIN18); no longer BPM1.18 (PIN17)
- net row4: now also BPM1.20 (PIN19); no longer BPM1.17 (PIN16)
- net row5: now also BPM1.21 (PIN20); no longer BPM1.16 (PIN15)
Changed lines of the file:
@@
 NoConn ~ 2100 3050
 NoConn ~ 2100 2950
+Text GLabel 2100 2350 0    50   Input ~ 0
+col5
+Text GLabel 2100 2450 0    50   Input ~ 0
+col4
 Text GLabel 2100 2850 0    50   Input ~ 0
-col5
+col3
 Text GLabel 2100 2750 0    50   Input ~ 0
-col4
+col2
 Text GLabel 2100 2650 0    50   Input ~ 0
-col3
+col1
 Text GLabel 2100 2550 0    50   Input ~ 0
-col2
-Text GLabel 2100 2450 0    50   Input ~ 0
-col1
-Text GLabel 2100 2350 0    50   Input ~ 0
 col0
+Text GLabel 3500 2850 2    50   Input ~ 0
+row0
+Text GLabel 3500 2750 2    50   Input ~ 0
+row1
+Text GLabel 3500 2650 2    50   Input ~ 0
+row2
+Text GLabel 3500 2550 2    50   Input ~ 0
+row3
+Text GLabel 3500 2450 2    50   Input ~ 0
+row4
 Text GLabel 3500 2350 2    50   Input ~ 0
-row0
-Text GLabel 3500 2450 2    50   Input ~ 0
-row1
-Text GLabel 3500 2550 2    50   Input ~ 0
-row2
-Text GLabel 3500 2650 2    50   Input ~ 0
-row3
-Text GLabel 3500 2750 2    50   Input ~ 0
-row4
-Text GLabel 3500 2850 2    50   Input ~ 0
 row5
 Text GLabel 8550 3000 0    50   Input ~ 0
